File: board/clock.kicad_sch (KiCad schematic)
At the start: 169 parts, among them J1 Conn_01x05_Pin, J2 Conn_01x05_Socket, J3 Barrel_Jack, Q1 Q_PNP, Q10 Q_NPN, Q11 Q_NPN, Q12 Q_NPN, Q13 Q_NPN, Q14 Q_NPN, Q15 Q_NPN, Q16 Q_NPN, Q17 Q_NPN, Q18 Q_NPN, Q19 Q_NPN, Q2 Q_PNP, Q20 Q_NPN, Q21 Q_NPN, Q22 Q_NPN, Q23 Q_NPN, Q24 Q_NPN, Q25 Q_NPN, Q26 Q_NPN, Q27 Q_NPN, Q28 Q_NPN, Q29 Q_NPN, Q3 Q_PNP, Q30 Q_NPN, Q31 Q_NPN, Q32 Q_NPN, Q33 Q_NPN, Q34 Q_NPN, Q35 Q_NPN, Q36 Q_NPN, Q37 Q_NPN, Q38 Q_NPN, Q39 Q_NPN, Q4 Q_PNP, Q40 Q_NPN, Q41 Q_NPN, Q42 Q_NPN, Q43 Q_NPN, Q44 Q_NPN, Q45 Q_NPN, Q5 Q_PNP, Q6 Q_PNP, Q7 Q_PNP, Q8 Q_NPN, Q9 Q_NPN, U1 ATmega328P-P, U10 DC56-11CGKWA, U11 DC56-11CGKWA, U12 DC56-11CGKWA, U13 DC56-11CGKWA, U14 DC56-11CGKWA, U15 DC56-11CGKWA, U16 DC56-11CGKWA, U17 DC56-11CGKWA, U18 DC56-11CGKWA, U19 DC56-11CGKWA, U2 74HC595, U20 DC56-11CGKWA, U21 DC56-11CGKWA, U22 DC56-11CGKWA, U23 DC56-11CGKWA, U24 DC56-11CGKWA, U25 DC56-11CGKWA, U26 DC56-11CGKWA, U27 DS1307+, U3 DC56-11CGKWA, U4 DC56-11CGKWA, U5 74HC595, U6 74HC595, U7 74HC595, U8 74HC595, U9 74HC595, Y1 16MHz, Y2 Crystal

Commit message: work
Parts:
- added RV1: 4kΩ, symbol Device:R_Potentiometer_US
- R10, R12, R14, R16, R18, R20, R22, R8: value R_US -> 470Ω
- R11, R13, R15, R17, R19, R21, R23, R9: value R_US -> 12Ω
- Y2: value Crystal -> 32.768kHz
Connections:
- net CTRL_DS1: now also U2.15 (QA)
- net CTRL_DS10: now also U5.1 (QB)
- net CTRL_DS11: now also U5.2 (QC)
- net CTRL_DS12: now also U5.3 (QD)
- net CTRL_DS13: now also U5.4 (QE)
- net CTRL_DS14: now also U5.5 (QF)
- net CTRL_DS15: now also U5.6 (QG)
- net CTRL_DS16: now also U5.7 (QH)
- net CTRL_DS17: now also U6.15 (QA)
- net CTRL_DS18: now also U6.1 (QB)
- net CTRL_DS19: now also U6.2 (QC)
- net CTRL_DS2: now also U2.1 (QB)
- net CTRL_DS20: now also U6.3 (QD)
- net CTRL_DS21: now also U6.4 (QE)
- net CTRL_DS22: now also U6.5 (QF)
- net CTRL_DS23: now also U6.6 (QG)
- net CTRL_DS24: now also U6.7 (QH)
- net CTRL_DS25: now also U7.15 (QA)
- net CTRL_DS26: now also U7.1 (QB)
- net CTRL_DS27: now also U7.2 (QC)
- net CTRL_DS28: now also U7.3 (QD)
- net CTRL_DS29: now also U7.4 (QE)
- net CTRL_DS3: now also U2.2 (QC)
- net CTRL_DS30: now also U7.5 (QF)
- net CTRL_DS31: now also U7.6 (QG)
- net CTRL_DS32: now also U7.7 (QH)
- net CTRL_DS33: now also U8.15 (QA)
- net CTRL_DS34: now also U8.1 (QB)
- net CTRL_DS35: now also U8.2 (QC)
- net CTRL_DS36: now also U8.3 (QD)
- net CTRL_DS37: now also U8.4 (QE)
- net CTRL_DS38: now also U8.5 (QF)
- net CTRL_DS4: now also U2.3 (QD)
- net CTRL_DS5: now also U2.4 (QE)
- net CTRL_DS6: now also U2.5 (QF)
- net CTRL_DS7: now also U2.6 (QG)
- net CTRL_DS8: now also U2.7 (QH)
- net CTRL_DS9: now also U5.15 (QA)
- net DS1: now also U3.13 (DIG2_CC); no longer U3.14 (DIG1_CC)
- net DS10: now also U12.14 (DIG1_CC); no longer U12.13 (DIG2_CC)
- net DS11: now also U13.13 (DIG2_CC); no longer U13.14 (DIG1_CC)
- net DS12: now also U13.14 (DIG1_CC); no longer U13.13 (DIG2_CC)
- net DS13: now also U14.13 (DIG2_CC); no longer U14.14 (DIG1_CC)
- net DS14: now also U14.14 (DIG1_CC); no longer U14.13 (DIG2_CC)
- net DS15: now also U21.13 (DIG2_CC); no longer U15.14 (DIG1_CC)
- net DS16: now also U21.14 (DIG1_CC); no longer U15.13 (DIG2_CC)
- net DS17: now also U20.13 (DIG2_CC); no longer U16.14 (DIG1_CC)
- net DS18: now also U20.14 (DIG1_CC); no longer U16.13 (DIG2_CC)
- net DS19: now also U19.13 (DIG2_CC); no longer U17.14 (DIG1_CC)
- net DS2: now also U3.14 (DIG1_CC); no longer U3.13 (DIG2_CC)
- net DS20: now also U19.14 (DIG1_CC); no longer U17.13 (DIG2_CC)
- net DS21: now also U18.13 (DIG2_CC); no longer U18.14 (DIG1_CC)
- net DS22: now also U18.14 (DIG1_CC); no longer U18.13 (DIG2_CC)
- net DS23: now also U17.13 (DIG2_CC); no longer U19.14 (DIG1_CC)
- net DS24: now also U17.14 (DIG1_CC); no longer U19.13 (DIG2_CC)
- net DS25: now also U16.13 (DIG2_CC); no longer U20.14 (DIG1_CC)
- net DS26: now also U16.14 (DIG1_CC); no longer U20.13 (DIG2_CC)
- net DS27: now also U15.13 (DIG2_CC); no longer U21.14 (DIG1_CC)
- net DS28: now also U15.14 (DIG1_CC); no longer U21.13 (DIG2_CC)
- net DS29: now also U24.13 (DIG2_CC); no longer U25.14 (DIG1_CC)
- net DS3: now also U4.13 (DIG2_CC); no longer U4.14 (DIG1_CC)
- net DS30: now also U24.14 (DIG1_CC); no longer U25.13 (DIG2_CC)
- net DS31: now also U23.13 (DIG2_CC); no longer U26.14 (DIG1_CC)
- net DS32: now also U23.14 (DIG1_CC); no longer U26.13 (DIG2_CC)
- net DS33: now also U22.13 (DIG2_CC); no longer U22.14 (DIG1_CC)
- net DS34: now also U22.14 (DIG1_CC); no longer U22.13 (DIG2_CC)
- net DS35: now also U26.13 (DIG2_CC); no longer U23.14 (DIG1_CC)
- net DS36: now also U26.14 (DIG1_CC); no longer U23.13 (DIG2_CC)
- net DS37: now also U25.13 (DIG2_CC); no longer U24.14 (DIG1_CC)
- net DS38: now also U25.14 (DIG1_CC); no longer U24.13 (DIG2_CC)
- net DS4: now also U4.14 (DIG1_CC); no longer U4.13 (DIG2_CC)
- net DS5: now also U10.13 (DIG2_CC); no longer U10.14 (DIG1_CC)
- net DS6: now also U10.14 (DIG1_CC); no longer U10.13 (DIG2_CC)
- net DS7: now also U11.13 (DIG2_CC); no longer U11.14 (DIG1_CC)
- net DS8: now also U11.14 (DIG1_CC); no longer U11.13 (DIG2_CC)
- net DS9: now also U12.13 (DIG2_CC); no longer U12.14 (DIG1_CC)
- net GND: now also RV1.3
- net VCC: now also RV1.1
- net BADJ: now reaches U1.23 (PC0)
- net BADJ: now also RV1.2
- no-connect marks 39 -> 54
Other:
- moved on the sheet: C1, C2, J1, R84, R85, U10, U11, U12, U13, U14, U3, U4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

Commit message: w
Parts:
- added C3, C4, C5, C6, C7, C8, C9: 22μF, symbol Device:C
- R24, R26, R28, R30, R32, R34, R36, R38, R40, R42, R44, R46, R48, R50, R52, R54, R56, R58, R60, R62, R64, R66, R68, R70, R72, R74, R76, R78, R80, R82: value R_US -> 470Ω
- R25, R27, R29, R31, R33, R35, R37, R39, R41, R43, R45, R47, R49, R51, R53, R55, R57, R59, R61, R63, R65, R67, R69, R71, R73, R75, R77, R79, R81, R83: value R_US -> 12Ω
Connections:
- net CTRL_DS18: now also R42.1; no longer R44.1
- net CTRL_DS19: now also R44.1; no longer R48.1
- net CTRL_DS20: now also R46.1; no longer R52.1
- net CTRL_DS21: now also R48.1; no longer R56.1
- net CTRL_DS22: now also R50.1; no longer R60.1
- net CTRL_DS23: now also R52.1; no longer R64.1
- net CTRL_DS24: now also R54.1; no longer R68.1
- net CTRL_DS25: now also R56.1; no longer R41.1
- net CTRL_DS26: now also R58.1; no longer R45.1
- net CTRL_DS27: now also R60.1; no longer R49.1
- net CTRL_DS28: now also R62.1; no longer R53.1
- net CTRL_DS29: now also R64.1; no longer R57.1
- net CTRL_DS30: now also R66.1; no longer R61.1
- net CTRL_DS31: now also R68.1; no longer R65.1
- net CTRL_DS32: now also R70.1; no longer R69.1
- net DS17: now also R41.1; no longer R42.1
- net DS18: now also R43.1; no longer R46.1
- net DS19: now also R45.1; no longer R50.1
- net DS20: now also R47.1; no longer R54.1
- net DS21: now also R49.1; no longer R58.1
- net DS22: now also R51.1; no longer R62.1
- net DS23: now also R53.1; no longer R66.1
- net DS24: now also R55.1; no longer R70.1
- net DS25: now also R57.1; no longer R43.1
- net DS26: now also R59.1; no longer R47.1
- net DS27: now also R61.1; no longer R51.1
- net DS28: now also R63.1; no longer R55.1
- net DS29: now also R65.1; no longer R59.1
- net DS30: now also R67.1; no longer R63.1
- net DS31: now also R69.1; no longer R67.1
- net GND: now also C3.2, C4.2, C5.2, C6.2, C7.2, C8.2, C9.2
- net VCC: now also C3.1, C4.1, C5.1, C6.1, C7.1, C8.1, C9.1
- net at Q34.B: now also R50.2; no longer R60.2
- net at Q31.B: now also R62.2; no longer R53.2
- net at Q31.C: now also R63.2; no longer R55.2
- net at Q24.C: now also R41.2; no longer R42.2
- net at Q34.C: now also R51.2; no longer R62.2
- net at Q38.B: now also R54.2; no longer R68.2
- net at Q38.C: now also R55.2; no longer R70.2
- net at R45.2: now also Q28.C; no longer Q27.B
- net at Q30.B: now also R46.2; no longer R52.2
- net at Q30.C: now also R47.2; no longer R54.2
- net at Q39.B: now also R70.2; no longer R69.2
- net at Q27.C: now also R59.2; no longer R47.2
- net at Q28.B: now also R44.2; no longer R48.2
- net at Q25.B: now also R56.2; no longer R41.2
- net at Q35.B: now also R66.2; no longer R61.2
- net at Q35.C: now also R67.2; no longer R63.2
- net at Q37.C: now also R69.2; no longer R67.2
- net at Q36.B: now also R52.2; no longer R64.2
- net at Q26.B: now also R42.2; no longer R44.2
- net at R57.2: now also Q25.C; no longer Q33.B
- net at R65.2: now also Q33.C; no longer Q37.B
- net at Q29.B: now also R60.2; no longer R49.2
- net at Q29.C: now also R61.2; no longer R51.2
- net at Q32.B: now also R48.2; no longer R56.2
- net at Q32.C: now also R49.2; no longer R58.2
- net at Q36.C: now also R53.2; no longer R66.2
- net at R43.2: now also Q26.C; no longer Q25.C
- new net: Q37.B, R68.2
- new net: Q33.B, R64.2
- new net: Q27.B, R58.2
Other:
- moved on the sheet: C1, C2, D1, D2, J3, Q1, Q10, Q11, Q12, Q13, Q14, Q15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
