File: old/clock.kicad_sch (KiCad schematic)
At the start: 177 parts, among them J1 Conn_01x05_Pin, J2 Conn_01x05_Socket, J3 Barrel_Jack, Q1 Q_PNP, Q10 Q_NPN, Q11 Q_NPN, Q12 Q_NPN, Q13 Q_NPN, Q14 Q_NPN, Q15 Q_NPN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

Commit message: old schematic
Parts:
- removed C1, C2: 22pF, symbol Device:C
- removed R84, R85: 10kΩ, symbol Device:R_US
