File: gps_enabled/clock.kicad_sch (KiCad schematic)
At the start: 177 parts, among them J1 Conn_01x05_Pin, J2 Conn_01x05_Socket, J3 Barrel_Jack, Q1 Q_PNP, Q10 Q_NPN, Q11 Q_NPN, Q12 Q_NPN, Q13 Q_NPN, Q14 Q_NPN, Q15 Q_NPN, Q16 Q_NPN, Q17 Q_NPN, Q18 Q_NPN, Q19 Q_NPN, Q2 Q_PNP, Q20 Q_NPN, Q21 Q_NPN, Q22 Q_NPN, Q23 Q_NPN, Q24 Q_NPN, Q25 Q_NPN, Q26 Q_NPN, Q27 Q_NPN, Q28 Q_NPN, Q29 Q_NPN, Q3 Q_PNP, Q30 Q_NPN, Q31 Q_NPN, Q32 Q_NPN, Q33 Q_NPN, Q34 Q_NPN, Q35 Q_NPN, Q36 Q_NPN, Q37 Q_NPN, Q38 Q_NPN, Q39 Q_NPN, Q4 Q_PNP, Q40 Q_NPN, Q41 Q_NPN, Q42 Q_NPN, Q43 Q_NPN, Q44 Q_NPN, Q45 Q_NPN, Q5 Q_PNP, Q6 Q_PNP, Q7 Q_PNP, Q8 Q_NPN, Q9 Q_NPN, U1 ATmega328P-P, U10 DC56-11CGKWA, U11 DC56-11CGKWA, U12 DC56-11CGKWA, U13 DC56-11CGKWA, U14 DC56-11CGKWA, U15 DC56-11CGKWA, U16 DC56-11CGKWA, U17 DC56-11CGKWA, U18 DC56-11CGKWA, U19 DC56-11CGKWA, U2 74HC595, U20 DC56-11CGKWA, U21 DC56-11CGKWA, U22 DC56-11CGKWA, U23 DC56-11CGKWA, U24 DC56-11CGKWA, U25 DC56-11CGKWA, U26 DC56-11CGKWA, U27 DS1307+, U3 DC56-11CGKWA, U4 DC56-11CGKWA, U5 74HC595, U6 74HC595, U7 74HC595, U8 74HC595, U9 74HC595, Y1 16MHz, Y2 32.768kHz

Commit message: w
Parts:
- added Q46: Q_PNP, Package_TO_SOT_THT:TO-220-3_Horizontal_TabDown, symbol Device:Q_PNP
- added R8: 10kΩ, Resistor_THT:R_Axial_DIN0207_L6.3mm_D2.5mm_P10.16mm_Horizontal, symbol Device:R_US
- added SW1: Increment, Button_Switch_THT:SW_PUSH_6mm, symbol Switch:SW_Push
- added SW2: Decrement, Button_Switch_THT:SW_PUSH_6mm, symbol Switch:SW_Push
- added SW3: Right, Button_Switch_THT:SW_PUSH_6mm, symbol Switch:SW_Push
- added SW4: Left, Button_Switch_THT:SW_PUSH_6mm, symbol Switch:SW_Push
- added SW5: Down, Button_Switch_THT:SW_PUSH_6mm, symbol Switch:SW_Push
- added SW6: Up, Button_Switch_THT:SW_PUSH_6mm, symbol Switch:SW_Push
- added SW7: Power, Button_Switch_THT:SW_Slide-03_Wuerth-WS-SLTV_10x2.5x6.4_P2.54mm, symbol Switch:SW_SPDT
- B1: renamed from BT1; value Battery_Cell -> 2032; footprint (none) -> Parts:BAT_BAT-HLD-001-THM
- C1, C2: footprint (none) -> Capacitor_SMD:C_1206_3216Metric_Pad1.33x1.80mm_HandSolder
- C3: footprint (none) -> Capacitor_THT:C_Radial_D5.0mm_H11.0mm_P2.00mm; symbol Device:C -> Device:C_Polarized_US
- C4: renamed from C9; footprint (none) -> Capacitor_THT:C_Radial_D5.0mm_H11.0mm_P2.00mm; symbol Device:C -> Device:C_Polarized_US
- C5: renamed from C4; footprint (none) -> Capacitor_THT:C_Radial_D5.0mm_H11.0mm_P2.00mm; symbol Device:C -> Device:C_Polarized_US
- C6: renamed from C5; footprint (none) -> Capacitor_THT:C_Radial_D5.0mm_H11.0mm_P2.00mm; symbol Device:C -> Device:C_Polarized_US
- C7: renamed from C6; footprint (none) -> Capacitor_THT:C_Radial_D5.0mm_H11.0mm_P2.00mm; symbol Device:C -> Device:C_Polarized_US
- C8: renamed from C7; footprint (none) -> Capacitor_THT:C_Radial_D5.0mm_H11.0mm_P2.00mm; symbol Device:C -> Device:C_Polarized_US
- C9: renamed from C8; footprint (none) -> Capacitor_THT:C_Radial_D5.0mm_H11.0mm_P2.00mm; symbol Device:C -> Device:C_Polarized_US
- D1, D2: footprint (none) -> LED_THT:LED_D5.0mm
- J1: renamed from J3; footprint (none) -> Connector_BarrelJack:BarrelJack_GCT_DCJ200-10-A_Horizontal
- J2: footprint (none) -> Connector_PinSocket_1.00mm:PinSocket_1x04_P1.00mm_Vertical
- J3: renamed from J1; footprint (none) -> Connector_PinHeader_1.00mm:PinHeader_1x04_P1.00mm_Vertical
- Q1, Q2, Q3, Q4, Q5, Q6, Q7: footprint (none) -> Package_TO_SOT_THT:TO-220-3_Horizontal_TabDown
- Q10, Q11, Q12, Q13, Q14, Q15, Q16, Q17, Q18, Q19, Q20, Q21, Q22, Q23, Q24, Q25, Q26, Q27, Q28, Q29, Q30, Q31, Q32, Q33, Q34, Q35, Q36, Q37, Q38, Q39, Q40, Q41, Q42, Q43, Q44, Q45, Q8, Q9: value Q_NPN -> 2N3904; footprint (none) -> Package_TO_SOT_THT:TO-92L_Inline
- R1, R2, R3, R4, R5, R6, R7: footprint (none) -> Resistor_THT:R_Axial_DIN0207_L6.3mm_D2.5mm_P10.16mm_Horizontal
- R10: renamed from R9; footprint (none) -> Resistor_THT:R_Axial_DIN0207_L6.3mm_D2.5mm_P10.16mm_Horizontal
- R11: renamed from R10; footprint (none) -> Resistor_THT:R_Axial_DIN0207_L6.3mm_D2.5mm_P10.16mm_Horizontal
- R12: renamed from R11; footprint (none) -> Resistor_THT:R_Axial_DIN0207_L6.3mm_D2.5mm_P10.16mm_Horizontal
- R13: renamed from R12; footprint (none) -> Resistor_THT:R_Axial_DIN0207_L6.3mm_D2.5mm_P10.16mm_Horizontal
- R14: renamed from R13; footprint (none) -> Resistor_THT:R_Axial_DIN0207_L6.3mm_D2.5mm_P10.16mm_Horizontal
- R15: renamed from R14; footprint (none) -> Resistor_THT:R_Axial_DIN0207_L6.3mm_D2.5mm_P10.16mm_Horizontal
- R16: renamed from R15; footprint (none) -> Resistor_THT:R_Axial_DIN0207_L6.3mm_D2.5mm_P10.16mm_Horizontal
- R17: renamed from R16; footprint (none) -> Resistor_THT:R_Axial_DIN0207_L6.3mm_D2.5mm_P10.16mm_Horizontal
- R18: renamed from R17; footprint (none) -> Resistor_THT:R_Axial_DIN0207_L6.3mm_D2.5mm_P10.16mm_Horizontal
- R19: renamed from R18; footprint (none) -> Resistor_THT:R_Axial_DIN0207_L6.3mm_D2.5mm_P10.16mm_Horizontal
- R20: renamed from R19; footprint (none) -> Resistor_THT:R_Axial_DIN0207_L6.3mm_D2.5mm_P10.16mm_Horizontal
- R21: renamed from R20; footprint (none) -> Resistor_THT:R_Axial_DIN0207_L6.3mm_D2.5mm_P10.16mm_Horizontal
- R22: renamed from R21; footprint (none) -> Resistor_THT:R_Axial_DIN0207_L6.3mm_D2.5mm_P10.16mm_Horizontal
- R23: renamed from R22; footprint (none) -> Resistor_THT:R_Axial_DIN0207_L6.3mm_D2.5mm_P10.16mm_Horizontal
- R24: renamed from R23; footprint (none) -> Resistor_THT:R_Axial_DIN0207_L6.3mm_D2.5mm_P10.16mm_Horizontal
- R25: renamed from R24; footprint (none) -> Resistor_THT:R_Axial_DIN0207_L6.3mm_D2.5mm_P10.16mm_Horizontal
- R26: renamed from R25; footprint (none) -> Resistor_THT:R_Axial_DIN0207_L6.3mm_D2.5mm_P10.16mm_Horizontal
- R27: renamed from R26; footprint (none) -> Resistor_THT:R_Axial_DIN0207_L6.3mm_D2.5mm_P10.16mm_Horizontal
- R28: renamed from R27; footprint (none) -> Resistor_THT:R_Axial_DIN0207_L6.3mm_D2.5mm_P10.16mm_Horizontal
- R29: renamed from R28; footprint (none) -> Resistor_THT:R_Axial_DIN0207_L6.3mm_D2.5mm_P10.16mm_Horizontal
- R30: renamed from R29; footprint (none) -> Resistor_THT:R_Axial_DIN0207_L6.3mm_D2.5mm_P10.16mm_Horizontal
- R31: renamed from R30; footprint (none) -> Resistor_THT:R_Axial_DIN0207_L6.3mm_D2.5mm_P10.16mm_Horizontal
- R32: renamed from R31; footprint (none) -> Resistor_THT:R_Axial_DIN0207_L6.3mm_D2.5mm_P10.16mm_Horizontal
- R33: renamed from R32; footprint (none) -> Resistor_THT:R_Axial_DIN0207_L6.3mm_D2.5mm_P10.16mm_Horizontal
- R34: renamed from R33; footprint (none) -> Resistor_THT:R_Axial_DIN0207_L6.3mm_D2.5mm_P10.16mm_Horizontal
- R35: renamed from R34; footprint (none) -> Resistor_THT:R_Axial_DIN0207_L6.3mm_D2.5mm_P10.16mm_Horizontal
- R36: renamed from R35; footprint (none) -> Resistor_THT:R_Axial_DIN0207_L6.3mm_D2.5mm_P10.16mm_Horizontal
- R37: renamed from R36; footprint (none) -> Resistor_THT:R_Axial_DIN0207_L6.3mm_D2.5mm_P10.16mm_Horizontal
- R38: renamed from R37; footprint (none) -> Resistor_THT:R_Axial_DIN0207_L6.3mm_D2.5mm_P10.16mm_Horizontal
- R39: renamed from R38; footprint (none) -> Resistor_THT:R_Axial_DIN0207_L6.3mm_D2.5mm_P10.16mm_Horizontal
- R40: renamed from R39; footprint (none) -> Resistor_THT:R_Axial_DIN0207_L6.3mm_D2.5mm_P10.16mm_Horizontal
- R41: renamed from R40; footprint (none) -> Resistor_THT:R_Axial_DIN0207_L6.3mm_D2.5mm_P10.16mm_Horizontal
- R42: renamed from R41; footprint (none) -> Resistor_THT:R_Axial_DIN0207_L6.3mm_D2.5mm_P10.16mm_Horizontal
- R43: renamed from R42; footprint (none) -> Resistor_THT:R_Axial_DIN0207_L6.3mm_D2.5mm_P10.16mm_Horizontal
- R44: renamed from R43; footprint (none) -> Resistor_THT:R_Axial_DIN0207_L6.3mm_D2.5mm_P10.16mm_Horizontal
- R45: renamed from R44; footprint (none) -> Resistor_THT:R_Axial_DIN0207_L6.3mm_D2.5mm_P10.16mm_Horizontal
- R46: renamed from R45; footprint (none) -> Resistor_THT:R_Axial_DIN0207_L6.3mm_D2.5mm_P10.16mm_Horizontal
- R47: renamed from R46; footprint (none) -> Resistor_THT:R_Axial_DIN0207_L6.3mm_D2.5mm_P10.16mm_Horizontal
- R48: renamed from R47; footprint (none) -> Resistor_THT:R_Axial_DIN0207_L6.3mm_D2.5mm_P10.16mm_Horizontal
- R49: renamed from R48; footprint (none) -> Resistor_THT:R_Axial_DIN0207_L6.3mm_D2.5mm_P10.16mm_Horizontal
- R50: renamed from R49; footprint (none) -> Resistor_THT:R_Axial_DIN0207_L6.3mm_D2.5mm_P10.16mm_Horizontal
- R51: renamed from R50; footprint (none) -> Resistor_THT:R_Axial_DIN0207_L6.3mm_D2.5mm_P10.16mm_Horizontal
- R52: renamed from R51; footprint (none) -> Resistor_THT:R_Axial_DIN0207_L6.3mm_D2.5mm_P10.16mm_Horizontal
- R53: renamed from R52; footprint (none) -> Resistor_THT:R_Axial_DIN0207_L6.3mm_D2.5mm_P10.16mm_Horizontal
- R54: renamed from R53; footprint (none) -> Resistor_THT:R_Axial_DIN0207_L6.3mm_D2.5mm_P10.16mm_Horizontal
- R55: renamed from R54; footprint (none) -> Resistor_THT:R_Axial_DIN0207_L6.3mm_D2.5mm_P10.16mm_Horizontal
- R56: renamed from R55; footprint (none) -> Resistor_THT:R_Axial_DIN0207_L6.3mm_D2.5mm_P10.16mm_Horizontal
- R57: renamed from R56; footprint (none) -> Resistor_THT:R_Axial_DIN0207_L6.3mm_D2.5mm_P10.16mm_Horizontal
- R58: renamed from R57; footprint (none) -> Resistor_THT:R_Axial_DIN0207_L6.3mm_D2.5mm_P10.16mm_Horizontal
- R59: renamed from R58; footprint (none) -> Resistor_THT:R_Axial_DIN0207_L6.3mm_D2.5mm_P10.16mm_Horizontal
- R60: renamed from R59; footprint (none) -> Resistor_THT:R_Axial_DIN0207_L6.3mm_D2.5mm_P10.16mm_Horizontal
- R61: renamed from R60; footprint (none) -> Resistor_THT:R_Axial_DIN0207_L6.3mm_D2.5mm_P10.16mm_Horizontal
- R62: renamed from R61; footprint (none) -> Resistor_THT:R_Axial_DIN0207_L6.3mm_D2.5mm_P10.16mm_Horizontal
- R63: renamed from R62; footprint (none) -> Resistor_THT:R_Axial_DIN0207_L6.3mm_D2.5mm_P10.16mm_Horizontal
- R64: renamed from R63; footprint (none) -> Resistor_THT:R_Axial_DIN0207_L6.3mm_D2.5mm_P10.16mm_Horizontal
- R65: renamed from R64; footprint (none) -> Resistor_THT:R_Axial_DIN0207_L6.3mm_D2.5mm_P10.16mm_Horizontal
- R66: renamed from R65; footprint (none) -> Resistor_THT:R_Axial_DIN0207_L6.3mm_D2.5mm_P10.16mm_Horizontal
- R67: renamed from R66; footprint (none) -> Resistor_THT:R_Axial_DIN0207_L6.3mm_D2.5mm_P10.16mm_Horizontal
- R68: renamed from R67; footprint (none) -> Resistor_THT:R_Axial_DIN0207_L6.3mm_D2.5mm_P10.16mm_Horizontal
- R69: renamed from R68; footprint (none) -> Resistor_THT:R_Axial_DIN0207_L6.3mm_D2.5mm_P10.16mm_Horizontal
- R70: renamed from R69; footprint (none) -> Resistor_THT:R_Axial_DIN0207_L6.3mm_D2.5mm_P10.16mm_Horizontal
- R71: renamed from R70; footprint (none) -> Resistor_THT:R_Axial_DIN0207_L6.3mm_D2.5mm_P10.16mm_Horizontal
- R72: renamed from R71; footprint (none) -> Resistor_THT:R_Axial_DIN0207_L6.3mm_D2.5mm_P10.16mm_Horizontal
- R73: renamed from R72; footprint (none) -> Resistor_THT:R_Axial_DIN0207_L6.3mm_D2.5mm_P10.16mm_Horizontal
- R74: renamed from R73; footprint (none) -> Resistor_THT:R_Axial_DIN0207_L6.3mm_D2.5mm_P10.16mm_Horizontal
- R75: renamed from R74; footprint (none) -> Resistor_THT:R_Axial_DIN0207_L6.3mm_D2.5mm_P10.16mm_Horizontal
- R76: renamed from R75; footprint (none) -> Resistor_THT:R_Axial_DIN0207_L6.3mm_D2.5mm_P10.16mm_Horizontal
- R77: renamed from R76; footprint (none) -> Resistor_THT:R_Axial_DIN0207_L6.3mm_D2.5mm_P10.16mm_Horizontal
- R78: renamed from R77; footprint (none) -> Resistor_THT:R_Axial_DIN0207_L6.3mm_D2.5mm_P10.16mm_Horizontal
- R79: renamed from R78; footprint (none) -> Resistor_THT:R_Axial_DIN0207_L6.3mm_D2.5mm_P10.16mm_Horizontal
- R80: renamed from R79; footprint (none) -> Resistor_THT:R_Axial_DIN0207_L6.3mm_D2.5mm_P10.16mm_Horizontal
- R81: renamed from R80; footprint (none) -> Resistor_THT:R_Axial_DIN0207_L6.3mm_D2.5mm_P10.16mm_Horizontal
- R82: renamed from R81; footprint (none) -> Resistor_THT:R_Axial_DIN0207_L6.3mm_D2.5mm_P10.16mm_Horizontal
- R83: renamed from R82; footprint (none) -> Resistor_THT:R_Axial_DIN0207_L6.3mm_D2.5mm_P10.16mm_Horizontal
- R84: renamed from R83; footprint (none) -> Resistor_THT:R_Axial_DIN0207_L6.3mm_D2.5mm_P10.16mm_Horizontal
- R85: renamed from R84; footprint (none) -> Resistor_THT:R_Axial_DIN0207_L6.3mm_D2.5mm_P10.16mm_Horizontal
- R86: renamed from R85; footprint (none) -> Resistor_THT:R_Axial_DIN0207_L6.3mm_D2.5mm_P10.16mm_Horizontal
- R87: renamed from R86; value R_US -> 470Ω; footprint (none) -> Resistor_THT:R_Axial_DIN0207_L6.3mm_D2.5mm_P10.16mm_Horizontal
- R88: renamed from R87; value R_US -> 470Ω; footprint (none) -> Resistor_THT:R_Axial_DIN0207_L6.3mm_D2.5mm_P10.16mm_Horizontal
- R9: renamed from R8; footprint (none) -> Resistor_THT:R_Axial_DIN0207_L6.3mm_D2.5mm_P10.16mm_Horizontal
- RV1: value 4kΩ -> 10kΩ; footprint (none) -> Potentiometer_THT:Potentiometer_Bourns_PTV09A-1_Single_Vertical
- U1: footprint Package_DIP:DIP-28_W7.62mm -> Package_DIP:DIP-28_W7.62mm_Socket_LongPads
- U2: renamed from U9; footprint (none) -> Package_DIP:DIP-16_W7.62mm_Socket_LongPads
- U3: renamed from U2; footprint (none) -> Package_DIP:DIP-16_W7.62mm_Socket_LongPads
- U4: renamed from U5; footprint (none) -> Package_DIP:DIP-16_W7.62mm_Socket_LongPads
- U5: renamed from U6; footprint (none) -> Package_DIP:DIP-16_W7.62mm_Socket_LongPads
- U6: renamed from U7; footprint (none) -> Package_DIP:DIP-16_W7.62mm_Socket_LongPads
- U7: renamed from U8; footprint (none) -> Package_DIP:DIP-16_W7.62mm_Socket_LongPads
- U8: renamed from U27; footprint Package_DIP:DIP-8_W7.62mm -> Package_DIP:DIP-8_W7.62mm_Socket_LongPads
- Y1: footprint (none) -> Crystal:Crystal_HC49-U_Vertical
- Y2: footprint (none) -> Crystal:Crystal_DS10_D1.0mm_L4.3mm_Vertical
- renumbered U3 to DS1, U19 to DS10, U18 to DS11, U17 to DS12, U16 to DS13, U15 to DS14, U24 to DS15, U23 to DS16, U22 to DS17, U26 to DS18, U25 to DS19, U4 to DS2, U10 to DS3, U11 to DS4, U12 to DS5, U13 to DS6, U14 to DS7, U21 to DS8, U20 to DS9
Connections:
- net DS37: no longer DS19.13 (DIG2_CC)
- net GND: now also SW1.1, SW2.1, SW3.1, SW4.1, SW5.1, SW6.1, SW7.2 (B)
- net VCC: now also Q46.E
- net DP: now reaches DS16.4 (DP1)
- net DP: now also DS1.4 (DP1), DS1.9 (DP2), DS10.4 (DP1), DS10.9 (DP2), DS11.4 (DP1), DS11.9 (DP2), DS12.4 (DP1), DS12.9 (DP2), DS13.4 (DP1), DS13.9 (DP2), DS14.4 (DP1), DS14.9 (DP2), DS15.4 (DP1), DS15.9 (DP2), DS16.9 (DP2), DS17.4 (DP1), DS17.9 (DP2), DS18.4 (DP1), DS18.9 (DP2), DS19.4 (DP1), DS19.9 (DP2), DS2.4 (DP1), DS2.9 (DP2), DS3.4 (DP1), DS3.9 (DP2), DS4.4 (DP1), DS4.9 (DP2), DS5.4 (DP1), DS5.9 (DP2), DS6.4 (DP1), DS6.9 (DP2), DS7.4 (DP1), DS7.9 (DP2), DS8.4 (DP1), DS8.9 (DP2), DS9.4 (DP1), DS9.9 (DP2), Q46.C
- net CTRL_DP: now reaches U2.7 (QH)
- net CTRL_DP: now also R8.1
- net RIGHT: now reaches U1.11 (PD5)
- net RIGHT: now also SW3.2
- net SET_ENABLE: now reaches U1.12 (PD6)
- net SET_ENABLE: now also SW7.1 (A)
- net INC: now reaches U1.2 (PD0)
- net INC: now also SW1.2
- net DEC: now reaches U1.3 (PD1)
- net DEC: now also SW2.2
- net UP: now reaches U1.4 (PD2)
- net UP: now also SW6.2
- net DOWN: now reaches U1.5 (PD3)
- net DOWN: now also SW5.2
- net LEFT: now reaches U1.6 (PD4)
- net LEFT: now also SW4.2
- new net: Q46.B, R8.2
- no-connect marks 54 -> 10
Other:
- moved on the sheet: Q1, Q2, Q3, Q4, Q5, Q6, Q7, R1, R2, R3, R4, R5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
