File: new/clock.kicad_pcb (KiCad board)
At the start: 2 copper layers, 186 parts, among them J1 Barrel_Jack, J2 Conn_01x05_Socket, J3 Conn_01x05_Pin, Q1 Q_PNP, Q10 2N3904, Q11 2N3904, Q12 2N3904, Q13 2N3904, Q14 2N3904, Q15 2N3904, Q16 2N3904, Q17 2N3904, Q18 2N3904, Q19 2N3904, Q2 Q_PNP, Q20 2N3904, Q21 2N3904, Q22 2N3904, Q23 2N3904, Q24 2N3904, Q25 2N3904, Q26 2N3904, Q27 2N3904, Q28 2N3904, Q29 2N3904, Q3 Q_PNP, Q30 2N3904, Q31 2N3904, Q32 2N3904, Q33 2N3904, Q34 2N3904, Q35 2N3904, Q36 2N3904, Q37 2N3904, Q38 2N3904, Q39 2N3904, Q4 Q_PNP, Q40 2N3904, Q41 2N3904, Q42 2N3904, Q43 2N3904, Q44 2N3904, Q45 2N3904, Q46 Q_PNP, Q5 Q_PNP, Q6 Q_PNP, Q7 Q_PNP, Q8 2N3904, Q9 2N3904, SW1 Increment, SW2 Decrement, SW3 Right, SW4 Left, SW5 Down, SW6 Up, SW7 Power, U1 ATmega328P-P, U2 74HC595, U3 74HC595, U4 74HC595, U5 74HC595, U6 74HC595, U7 74HC595, U8 DS1307+, Y1 16MHz, Y2 32.768kHz

Commit message: work
Parts:
- added D3: TVS, Diode_SMD:D_SMA_Handsoldering, F.Cu at (58.5, 155.5)
- added SW8: Power, Button_Switch_THT:SW_Slide-03_Wuerth-WS-SLTV_10x2.5x6.4_P2.54mm, F.Cu at (58.0, 150.5)
- DS1, DS10, DS11, DS12, DS13, DS14, DS15, DS16, DS17, DS18, DS19, DS2, DS3, DS4, DS5, DS6, DS7, DS8, DS9: footprint Display_7Segment:DA56-11CGKWA -> Parts:DIPS2200W51P254L3580H1000Q18N
- J2: footprint Connector_PinSocket_1.00mm:PinSocket_1x04_P1.00mm_Vertical -> Connector_PinSocket_2.54mm:PinSocket_1x05_P2.54mm_Vertical
- J3: footprint Connector_PinHeader_1.00mm:PinHeader_1x04_P1.00mm_Vertical -> Connector_PinHeader_2.54mm:PinHeader_1x05_P2.54mm_Vertical
- Q1, Q2, Q3, Q4, Q5, Q6, Q7: value Q_PNP -> TIP127
- Q8: renamed from Q46; value Q_PNP -> TIP127
- SW7: value Power -> Set
- moved U2 434.6 mm to (488.2, 83.6)
- moved U3 415.9 mm to (480.9, 83.2), turned to -90 degrees
- moved U4 401.6 mm to (480.9, 102.4), turned to -90 degrees
- moved J3 400.8 mm to (540.6, 144.4)
- moved U8 396.1 mm to (525.0, 141.9)
- moved U5 388.1 mm to (480.9, 121.4), turned to -90 degrees
- moved Y2 380.3 mm to (526.1, 154.9)
- moved U6 375.5 mm to (480.9, 140.5), turned to -90 degrees
- moved U7 363.8 mm to (480.9, 158.4), turned to -90 degrees
- moved C1 354.1 mm to (494.5, 120.0)
- moved J2 351.4 mm to (488.5, 106.4)
- moved C2 348.4 mm to (488.5, 120.0)
- moved Q8 346.6 mm to (479.5, 72.7)
- moved Q7 345.1 mm to (466.5, 72.7)
- moved Q6 343.7 mm to (453.5, 72.7)
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- renumbered Q9 to Q10, Q10 to Q11, Q11 to Q12, Q12 to Q13, Q13 to Q14, Q14 to Q15, Q15 to Q16, Q16 to Q17, Q17 to Q18, Q18 to Q19, Q19 to Q20, Q20 to Q21, Q21 to Q22, Q22 to Q23, Q23 to Q24, Q24 to Q25, Q28 to Q27, Q30 to Q28, Q32 to Q29, Q34 to Q30, Q36 to Q31, Q38 to Q32, Q25 to Q33, Q27 to Q34, Q29 to Q35, Q31 to Q36, Q33 to Q37, Q35 to Q38, Q37 to Q39, Q39 to Q40, Q40 to Q41, Q41 to Q42, Q42 to Q43, Q43 to Q44, Q44 to Q45, Q45 to Q46, Q8 to Q9
Connections:
- J1 pad 1: VCC -> Net-(SW8-B)
- Q1 pad 1: (no net) -> Net-(Q1-PadC)
- Q1 pad 2: (no net) -> DIG_A
- Q1 pad 3: (no net) -> VCC
- Q10 pad 1: (no net) -> GND
- Q10 pad 2: (no net) -> Net-(Q10-B)
- Q10 pad 3: (no net) -> Net-(Q10-C)
- Q11 pad 1: (no net) -> GND
- Q11 pad 2: (no net) -> Net-(Q11-B)
- Q11 pad 3: (no net) -> Net-(Q11-C)
- Q12 pad 1: (no net) -> GND
- Q12 pad 2: (no net) -> Net-(Q12-B)
- Q12 pad 3: (no net) -> Net-(Q12-C)
- Q13 pad 1: (no net) -> GND
- Q13 pad 2: (no net) -> Net-(Q13-B)
- Q13 pad 3: (no net) -> Net-(Q13-C)
- Q14 pad 1: (no net) -> GND
- Q14 pad 2: (no net) -> Net-(Q14-B)
- Q14 pad 3: (no net) -> Net-(Q14-C)
- Q15 pad 1: (no net) -> GND
- Q15 pad 2: (no net) -> Net-(Q15-B)
- Q15 pad 3: (no net) -> Net-(Q15-C)
- Q16 pad 1: (no net) -> GND
- Q16 pad 2: (no net) -> Net-(Q16-B)
- Q16 pad 3: (no net) -> Net-(Q16-C)
- Q17 pad 1: (no net) -> GND
- Q17 pad 2: (no net) -> Net-(Q17-B)
- Q17 pad 3: (no net) -> Net-(Q17-C)
- Q18 pad 1: (no net) -> GND
- Q18 pad 2: (no net) -> Net-(Q18-B)
- Q18 pad 3: (no net) -> Net-(Q18-C)
- Q19 pad 1: (no net) -> GND
- Q19 pad 2: (no net) -> Net-(Q19-B)
- Q19 pad 3: (no net) -> Net-(Q19-C)
- Q2 pad 1: (no net) -> Net-(Q2-PadE)
- Q2 pad 2: (no net) -> DIG_B
- Q2 pad 3: (no net) -> VCC
- Q20 pad 1: (no net) -> GND
- Q20 pad 2: (no net) -> Net-(Q20-B)
- Q20 pad 3: (no net) -> Net-(Q20-C)
- Q21 pad 1: (no net) -> GND
- Q21 pad 2: (no net) -> Net-(Q21-B)
- Q21 pad 3: (no net) -> Net-(Q21-C)
- Q22 pad 1: (no net) -> GND
- Q22 pad 2: (no net) -> Net-(Q22-B)
- Q22 pad 3: (no net) -> Net-(Q22-C)
- Q23 pad 1: (no net) -> GND
- Q23 pad 2: (no net) -> Net-(Q23-B)
- Q23 pad 3: (no net) -> Net-(Q23-C)
- Q24 pad 1: (no net) -> GND
- Q24 pad 2: (no net) -> Net-(Q24-B)
- Q24 pad 3: (no net) -> Net-(Q24-C)
- Q25 pad 1: (no net) -> GND
- Q25 pad 2: (no net) -> Net-(Q25-B)
- Q25 pad 3: (no net) -> Net-(Q25-C)
- Q26 pad 1: (no net) -> GND
- Q26 pad 2: (no net) -> Net-(Q26-B)
- Q26 pad 3: (no net) -> Net-(Q26-C)
- Q27 pad 1: (no net) -> GND
- Q27 pad 2: (no net) -> Net-(Q27-B)
- Q27 pad 3: (no net) -> Net-(Q27-C)
- Q28 pad 1: (no net) -> GND
- Q28 pad 2: (no net) -> Net-(Q28-B)
- Q28 pad 3: (no net) -> Net-(Q28-C)
- Q29 pad 1: (no net) -> GND
- Q29 pad 2: (no net) -> Net-(Q29-B)
- Q29 pad 3: (no net) -> Net-(Q29-C)
- Q3 pad 1: (no net) -> Net-(Q3-PadB)
- Q3 pad 2: (no net) -> DIG_C
- Q3 pad 3: (no net) -> VCC
- Q30 pad 1: (no net) -> GND
- Q30 pad 2: (no net) -> Net-(Q30-B)
- Q30 pad 3: (no net) -> Net-(Q30-C)
- Q31 pad 1: (no net) -> GND
- Q31 pad 2: (no net) -> Net-(Q31-B)
- Q31 pad 3: (no net) -> Net-(Q31-C)
- Q32 pad 1: (no net) -> GND
- Q32 pad 2: (no net) -> Net-(Q32-B)
- Q32 pad 3: (no net) -> Net-(Q32-C)
- Q33 pad 1: (no net) -> GND
- Q33 pad 2: (no net) -> Net-(Q33-B)
- Q33 pad 3: (no net) -> Net-(Q33-C)
- Q34 pad 1: (no net) -> GND
- Q34 pad 2: (no net) -> Net-(Q34-B)
- Q34 pad 3: (no net) -> Net-(Q34-C)
- Q35 pad 1: (no net) -> GND
- Q35 pad 2: (no net) -> Net-(Q35-B)
- Q35 pad 3: (no net) -> Net-(Q35-C)
- Q36 pad 1: (no net) -> GND
- Q36 pad 2: (no net) -> Net-(Q36-B)
- Q36 pad 3: (no net) -> Net-(Q36-C)
- Q37 pad 1: (no net) -> GND
- Q37 pad 2: (no net) -> Net-(Q37-B)
- Q37 pad 3: (no net) -> Net-(Q37-C)
- Q38 pad 1: (no net) -> GND
- Q38 pad 2: (no net) -> Net-(Q38-B)
- Q38 pad 3: (no net) -> Net-(Q38-C)
- Q39 pad 1: (no net) -> GND
- Q39 pad 2: (no net) -> Net-(Q39-B)
- Q39 pad 3: (no net) -> Net-(Q39-C)
- Q4 pad 1: (no net) -> Net-(Q4-PadE)
- Q4 pad 2: (no net) -> DIG_D
- Q4 pad 3: (no net) -> VCC
- Q40 pad 1: (no net) -> GND
- Q40 pad 2: (no net) -> Net-(Q40-B)
- Q40 pad 3: (no net) -> Net-(Q40-C)
- Q41 pad 1: (no net) -> GND
- Q41 pad 2: (no net) -> Net-(Q41-B)
- Q41 pad 3: (no net) -> Net-(Q41-C)
- Q42 pad 1: (no net) -> GND
- Q42 pad 2: (no net) -> Net-(Q42-B)
- Q42 pad 3: (no net) -> Net-(Q42-C)
- Q43 pad 1: (no net) -> GND
- Q43 pad 2: (no net) -> Net-(Q43-B)
- Q43 pad 3: (no net) -> Net-(Q43-C)
- Q44 pad 1: (no net) -> GND
- Q44 pad 2: (no net) -> Net-(Q44-B)
- Q44 pad 3: (no net) -> Net-(Q44-C)
- Q45 pad 1: (no net) -> GND
- Q45 pad 2: (no net) -> Net-(Q45-B)
- Q45 pad 3: (no net) -> Net-(Q45-C)
- Q46 pad 1: (no net) -> GND
- Q46 pad 2: (no net) -> Net-(Q46-B)
- Q46 pad 3: (no net) -> Net-(Q46-C)
- Q5 pad 1: (no net) -> Net-(Q5-PadB)
- Q5 pad 2: (no net) -> DIG_E
- Q5 pad 3: (no net) -> VCC
- Q6 pad 1: (no net) -> Net-(Q6-PadC)
- Q6 pad 2: (no net) -> DIG_F
- Q6 pad 3: (no net) -> VCC
- Q7 pad 1: (no net) -> Net-(Q7-PadE)
- Q7 pad 2: (no net) -> DIG_G
- Q7 pad 3: (no net) -> VCC
- Q8 pad 1: (no net) -> Net-(Q8-B)
- Q8 pad 2: (no net) -> DP
- Q8 pad 3: (no net) -> VCC
- Q9 pad 1: (no net) -> GND
- Q9 pad 2: (no net) -> Net-(Q9-B)
- Q9 pad 3: (no net) -> Net-(Q9-C)
- R1 pad 2: Net-(Q1-PadB) -> Net-(Q1-PadC)
- R10 pad 2: Net-(Q8-PadC) -> Net-(Q9-C)
- R11 pad 2: Net-(Q9-PadB) -> Net-(Q10-B)
- R12 pad 2: Net-(Q9-PadC) -> Net-(Q10-C)
- R13 pad 2: Net-(Q10-PadB) -> Net-(Q11-B)
- R14 pad 2: Net-(Q10-PadC) -> Net-(Q11-C)
- R15 pad 2: Net-(Q11-PadB) -> Net-(Q12-B)
- R16 pad 2: Net-(Q11-PadC) -> Net-(Q12-C)
- R17 pad 2: Net-(Q12-PadB) -> Net-(Q13-B)
- R18 pad 2: Net-(Q12-PadC) -> Net-(Q13-C)
- R19 pad 2: Net-(Q13-PadB) -> Net-(Q14-B)
- R2 pad 2: Net-(Q2-PadB) -> Net-(Q2-PadE)
- R20 pad 2: Net-(Q13-PadC) -> Net-(Q14-C)
- R21 pad 2: Net-(Q14-PadB) -> Net-(Q15-B)
- R22 pad 2: Net-(Q14-PadC) -> Net-(Q15-C)
- R23 pad 2: Net-(Q15-PadB) -> Net-(Q16-B)
- R24 pad 2: Net-(Q15-PadC) -> Net-(Q16-C)
- R25 pad 2: Net-(Q16-PadB) -> Net-(Q17-B)
- R26 pad 2: Net-(Q16-PadC) -> Net-(Q17-C)
- R27 pad 2: Net-(Q17-PadB) -> Net-(Q18-B)
- R28 pad 2: Net-(Q17-PadC) -> Net-(Q18-C)
- R29 pad 2: Net-(Q18-PadB) -> Net-(Q19-B)
- R30 pad 2: Net-(Q18-PadC) -> Net-(Q19-C)
- R31 pad 2: Net-(Q19-PadB) -> Net-(Q20-B)
- R32 pad 2: Net-(Q19-PadC) -> Net-(Q20-C)
- R33 pad 2: Net-(Q20-PadB) -> Net-(Q21-B)
- R34 pad 2: Net-(Q20-PadC) -> Net-(Q21-C)
- R35 pad 2: Net-(Q21-PadB) -> Net-(Q22-B)
- R36 pad 2: Net-(Q21-PadC) -> Net-(Q22-C)
- R37 pad 2: Net-(Q22-PadB) -> Net-(Q23-B)
- R38 pad 2: Net-(Q22-PadC) -> Net-(Q23-C)
- R39 pad 2: Net-(Q23-PadB) -> Net-(Q24-B)
- R4 pad 2: Net-(Q4-PadB) -> Net-(Q4-PadE)
- R40 pad 2: Net-(Q23-PadC) -> Net-(Q24-C)
- R41 pad 2: Net-(Q24-PadB) -> Net-(Q25-B)
- R42 pad 2: Net-(Q24-PadC) -> Net-(Q25-C)
- R43 pad 2: Net-(Q26-PadB) -> Net-(Q26-B)
- R44 pad 2: Net-(Q26-PadC) -> Net-(Q26-C)
- R45 pad 2: Net-(Q28-PadB) -> Net-(Q27-B)
- R46 pad 2: Net-(Q28-PadC) -> Net-(Q27-C)
- R47 pad 2: Net-(Q30-PadB) -> Net-(Q28-B)
- R48 pad 2: Net-(Q30-PadC) -> Net-(Q28-C)
- R49 pad 2: Net-(Q32-PadB) -> Net-(Q29-B)
- R50 pad 2: Net-(Q32-PadC) -> Net-(Q29-C)
- R51 pad 2: Net-(Q34-PadB) -> Net-(Q30-B)
- R52 pad 2: Net-(Q34-PadC) -> Net-(Q30-C)
- R53 pad 2: Net-(Q36-PadB) -> Net-(Q31-B)
- R54 pad 2: Net-(Q36-PadC) -> Net-(Q31-C)
- R55 pad 2: Net-(Q38-PadB) -> Net-(Q32-B)
- R56 pad 2: Net-(Q38-PadC) -> Net-(Q32-C)
- R57 pad 2: Net-(Q25-PadB) -> Net-(Q33-B)
- R58 pad 2: Net-(Q25-PadC) -> Net-(Q33-C)
- R59 pad 2: Net-(Q27-PadB) -> Net-(Q34-B)
- R6 pad 2: Net-(Q6-PadB) -> Net-(Q6-PadC)
- R60 pad 2: Net-(Q27-PadC) -> Net-(Q34-C)
- R61 pad 2: Net-(Q29-PadB) -> Net-(Q35-B)
- R62 pad 2: Net-(Q29-PadC) -> Net-(Q35-C)
- R63 pad 2: Net-(Q31-PadB) -> Net-(Q36-B)
- R64 pad 2: Net-(Q31-PadC) -> Net-(Q36-C)
- R65 pad 2: Net-(Q33-PadB) -> Net-(Q37-B)
- R66 pad 2: Net-(Q33-PadC) -> Net-(Q37-C)
- R67 pad 2: Net-(Q35-PadB) -> Net-(Q38-B)
- R68 pad 2: Net-(Q35-PadC) -> Net-(Q38-C)
- R69 pad 2: Net-(Q37-PadB) -> Net-(Q39-B)
- R7 pad 2: Net-(Q7-PadB) -> Net-(Q7-PadE)
- R70 pad 2: Net-(Q37-PadC) -> Net-(Q39-C)
- R71 pad 2: Net-(Q39-PadB) -> Net-(Q40-B)
- R72 pad 2: Net-(Q39-PadC) -> Net-(Q40-C)
- R73 pad 2: Net-(Q40-PadB) -> Net-(Q41-B)
- R74 pad 2: Net-(Q40-PadC) -> Net-(Q41-C)
- R75 pad 2: Net-(Q41-PadB) -> Net-(Q42-B)
- R76 pad 2: Net-(Q41-PadC) -> Net-(Q42-C)
- R77 pad 2: Net-(Q42-PadB) -> Net-(Q43-B)
- R78 pad 2: Net-(Q42-PadC) -> Net-(Q43-C)
- R79 pad 2: Net-(Q43-PadB) -> Net-(Q44-B)
- R8 pad 2: Net-(Q46-PadB) -> Net-(Q8-B)
- R80 pad 2: Net-(Q43-PadC) -> Net-(Q44-C)
- R81 pad 2: Net-(Q44-PadB) -> Net-(Q45-B)
- R82 pad 2: Net-(Q44-PadC) -> Net-(Q45-C)
- R83 pad 2: Net-(Q45-PadB) -> Net-(Q46-B)
- R84 pad 2: Net-(Q45-PadC) -> Net-(Q46-C)
- R9 pad 2: Net-(Q8-PadB) -> Net-(Q9-B)
Other:
- board outline added: 450 x 120 mm

Commit message: w
Parts:
- moved R86 152.7 mm to (498.0, 116.1), turned to 90 degrees
- moved R85 146.7 mm to (493.4, 116.1), turned to 90 degrees
- moved R84 106.4 mm to (481.8, 154.4), turned to 180 degrees
- moved R83 100.6 mm to (481.8, 158.5), turned to 180 degrees
- moved Q46 96.7 mm to (465.8, 154.4)
- moved R82 95.1 mm to (481.9, 162.9), turned to 180 degrees
- moved R81 90.1 mm to (481.9, 167.0), turned to 180 degrees
- moved Q45 88.8 mm to (465.8, 163.0)
- moved R80 75.0 mm to (462.2, 162.9), turned to 180 degrees
- moved R79 69.6 mm to (462.2, 167.0), turned to 180 degrees
- moved Q44 69.3 mm to (446.2, 163.0)
- moved R78 56.1 mm to (442.9, 163.0), turned to 180 degrees
- moved Q43 50.4 mm to (426.8, 163.0)
- moved R77 49.9 mm to (442.9, 167.1), turned to 180 degrees
- moved R76 39.4 mm to (423.4, 162.9), turned to 180 degrees
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Routing:
- net DIG_G: track 0.00 -> 1327.2 mm
- net DP: track 0.00 -> 1063.5 mm
- net DIG_C: track 0.00 -> 1044.7 mm
- net DIG_D: track 0.00 -> 1027.5 mm
- net DIG_E: track 0.00 -> 1019.1 mm
- net DIG_F: track 0.00 -> 965.8 mm
- net DIG_A: track 0.00 -> 945.2 mm
- net DIG_B: track 0.00 -> 932.6 mm
- net RCLK: track 0.00 -> 192.9 mm
- net ~{OE}: track 0.00 -> 161.5 mm
- net CTRL_DS26: track 0.00 -> 122.7 mm, vias 0 -> 1
- net CTRL_DS27: track 0.00 -> 112.0 mm, vias 0 -> 2
- net CTRL_DS18: track 0.00 -> 111.9 mm
- net DCLK: track 0.00 -> 108.7 mm
- net CTRL_DS17: track 0.00 -> 107.7 mm, vias 0 -> 1
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- added copper zone on F.Cu, net GND
- added copper zone on B.Cu, net VCC
Other:
- copper layers 2 -> 4

Commit message: huge
Parts:
- moved Y2 52.0 mm to (551.4, 109.5)
- moved U8 50.0 mm to (548.3, 96.2)
- moved J3 46.1 mm to (562.1, 99.2)
- moved B1 25.4 mm to (535.5, 105.0), turned to -90 degrees
- moved R73 0.70 mm to (403.9, 167.8)
- moved R75 0.70 mm to (423.4, 167.7)
- moved R77 0.70 mm to (442.9, 167.8)
- moved R79 0.70 mm to (462.2, 167.7)
Connections:
- DS19 pad 13: unconnected-(DS19-DIG2_CC-Pad13) -> DS37
Routing:
- net DP: track 1063.5 -> 1526.8 mm
- net DIG_E: track 1019.1 -> 1449.7 mm, vias 0 -> 1
- net DS14: track 0.00 -> 416.8 mm, vias 0 -> 2
- net DIG_D: track 1027.5 -> 1443.1 mm, vias 0 -> 1
- net DS13: track 0.00 -> 405.0 mm, vias 0 -> 2
- net DS28: track 0.00 -> 400.1 mm, vias 0 -> 2
- net DIG_C: track 1044.7 -> 1442.5 mm
- net DS27: track 0.00 -> 388.9 mm, vias 0 -> 2
- net DS12: track 0.00 -> 361.8 mm, vias 0 -> 2
- net DS11: track 0.00 -> 350.4 mm, vias 0 -> 2
- net DS26: track 0.00 -> 345.2 mm, vias 0 -> 2
- net DS25: track 0.00 -> 333.9 mm, vias 0 -> 2
- net DS38: track 0.00 -> 332.1 mm, vias 0 -> 2
- net DS24: track 0.00 -> 329.1 mm, vias 0 -> 2
- net DS37: track 0.00 -> 328.6 mm, vias 0 -> 1
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Other:
- board size 450 x 120 mm -> 515.5 x 120 mm

Commit message: work
Parts:
- moved R81 0.75 mm to (481.9, 167.8)
- moved Q46 0.45 mm to (465.8, 154.0)
- moved R84 0.45 mm to (481.8, 154.0)
Routing:
- net INC: track 6.50 -> 467.6 mm
- net UP: track 6.50 -> 460.5 mm, vias 0 -> 1
- net DEC: track 6.50 -> 459.0 mm, vias 0 -> 1
- net LEFT: track 6.50 -> 437.0 mm
- net DOWN: track 6.50 -> 423.8 mm, vias 0 -> 1
- net RIGHT: track 6.50 -> 400.1 mm, vias 0 -> 1
- net SET_ENABLE: track 0.00 -> 372.5 mm, vias 0 -> 3
- net BADJ: track 0.00 -> 369.3 mm, vias 0 -> 3
- net CTRL_DS36: track 68.3 -> 66.2 mm, vias 0 -> 1
- net DCLK: track 108.7 -> 107.4 mm, vias 0 -> 1
- net ~{OE}: track 161.5 -> 160.4 mm
- net CTRL_DS37: track 46.7 -> 47.4 mm
- net SCLK: track 74.2 -> 74.9 mm, vias 0 -> 1

Commit message: almost
Parts:
- added J4: Conn_PIC_ICSP_ICD, Connector_IDC:IDC-Header_2x03_P2.54mm_Vertical, F.Cu at (467.2, 146.5)
- moved J3 49.3 mm to (537.1, 56.8)
- moved U8 49.3 mm to (523.2, 53.8)
- moved Y2 49.3 mm to (526.3, 67.1)
- moved B1 49.3 mm to (510.4, 62.6)
- moved J1 2.45 mm to (64.3, 162.8)
Connections:
- U1 pad 1: unconnected-(U1-~{RESET}/PC6-Pad1) -> RESET
- U1 pad 19: unconnected-(U1-PB5-Pad19) -> SCK
Routing:
- net SCK: track 0.00 -> 55.7 mm, vias 0 -> 2
- net SER: track 95.8 -> 144.7 mm, vias 0 -> 1
- net RESET: track 0.00 -> 23.7 mm, vias 0 -> 2
- net RCLK: track 192.9 -> 201.9 mm
- net Net-(SW8-B): track 12.9 -> 15.3 mm
- net CTRL_DS33: track 93.8 -> 95.2 mm
- net CTRL_DS34: track 89.9 -> 91.2 mm
- net CTRL_DS35: track 75.0 -> 76.2 mm
- net DOWN: track 423.8 -> 424.7 mm
- net DIG_G: vias 0 -> 1
- net DCLK: vias 1 -> 2
Other:
- board size 515.5 x 120 mm -> 490.4 x 120 mm
- board text added: "2032"
