File: new/clock.kicad_pcb (KiCad board)
At the start: 4 copper layers, 490.4 x 120 mm, 189 parts, among them J1 Barrel_Jack, J2 Conn_01x05_Socket, J3 Conn_01x05_Pin, J4 Conn_PIC_ICSP_ICD, Q1 TIP127, Q10 2N3904, Q11 2N3904, Q12 2N3904, Q13 2N3904, Q14 2N3904, Q15 2N3904, Q16 2N3904, Q17 2N3904, Q18 2N3904, Q19 2N3904, Q2 TIP127, Q20 2N3904, Q21 2N3904, Q22 2N3904, Q23 2N3904, Q24 2N3904, Q25 2N3904, Q26 2N3904, Q27 2N3904, Q28 2N3904, Q29 2N3904, Q3 TIP127, Q30 2N3904, Q31 2N3904, Q32 2N3904, Q33 2N3904, Q34 2N3904, Q35 2N3904, Q36 2N3904, Q37 2N3904, Q38 2N3904, Q39 2N3904, Q4 TIP127, Q40 2N3904, Q41 2N3904, Q42 2N3904, Q43 2N3904, Q44 2N3904, Q45 2N3904, Q46 2N3904, Q5 TIP127, Q6 TIP127, Q7 TIP127, Q8 TIP127, Q9 2N3904, SW1 Increment, SW2 Decrement, SW3 Right, SW4 Left, SW5 Down, SW6 Up, SW7 Set, SW8 Power, U1 ATmega328P-P, U2 74HC595, U3 74HC595, U4 74HC595, U5 74HC595, U6 74HC595, U7 74HC595, U8 DS1307+, Y1 16MHz, Y2 32.768kHz

Commit message: done?
Parts:
- removed the J3 at (537.1, 56.8)
- added SW9: Set, Button_Switch_THT:SW_Slide-03_Wuerth-WS-SLTV_10x2.5x6.4_P2.54mm, F.Cu at (57.8, 133.5)
- B1: moved to B.Cu
- moved B1 180.1 mm to (330.5, 70.8), turned to 0 degrees
- moved Y2 36.1 mm to (491.0, 74.8), turned to 180 degrees
- moved U8 34.7 mm to (489.7, 62.7)
- moved SW8 16.0 mm to (131.2, 159.0), turned to 180 degrees
- moved RV1 7.75 mm to (133.8, 151.8)
- moved C4 6.25 mm to (494.2, 78.5)
- renumbered J4 to J3, SW8 to SW1, SW1 to SW2, SW2 to SW3, SW6 to SW4, SW4 to SW6, SW3 to SW7, SW7 to SW8
Connections:
- B1 pad 2: Net-(B1--) -> GND
- U1 pad 13: unconnected-(U1-PD7-Pad13) -> Mode
- U8 pad 4: Net-(B1--) -> GND
- U8 pad 5: Net-(J3-Pin_4) -> SDA
- U8 pad 6: Net-(J3-Pin_3) -> SCL
- U8 pad 7: Net-(J3-Pin_2) -> unconnected-(U8-SQW/OUT-Pad7)
- U8 pad 8: Net-(J3-Pin_1) -> VCC
Routing:
- net Mode: track 0.00 -> 466.0 mm, vias 0 -> 2
- net Net-(B1-+): track 43.6 -> 216.0 mm, vias 0 -> 2
- net SCL: track 32.5 -> 72.9 mm
- net SDA: track 38.2 -> 75.2 mm
- net Net-(B1--): track 29.5 -> 0.00 mm
- net SET_ENABLE: track 372.5 -> 364.3 mm
- net BADJ: track 369.3 -> 376.9 mm
- net Net-(J3-Pin_4): track 7.46 -> 0.00 mm
- net Net-(J3-Pin_3): track 7.46 -> 0.00 mm
- net Net-(J3-Pin_2): track 7.46 -> 0.00 mm
- net Net-(J3-Pin_1): track 7.46 -> 0.00 mm
- net Net-(U8-X1): track 15.2 -> 21.1 mm
- net SCLK: track 74.9 -> 73.1 mm, vias 1 -> 0
- net DS16: track 116.4 -> 115.1 mm
- net RIGHT: track 400.1 -> 399.1 mm
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Other:
- board size 490.4 x 120 mm -> 450 x 120 mm
- board text added: "AM/PM"
- board text added: "Bright"
- board text added: "Brightness"
- board text added: "Current Time"
- board text added: "Day"
- board text added: "Days"
- board text added: "Designed by Kyle Schmerge in association with UCSB IEEE. www.github.com/kpzip www.ucsbieee.org"
- board text added: "Difference"
- board text added: "Dim"
- board text added: "Down"
- board text added: "EXT CLK"
- board text added: "Hour"
- board text added: "Hours"
- board text added: "Left"
- board text added: "Lock"
- board text added: "Minute"
- board text added: "Minutes"
- board text added: "Month"
- board text added: "Off"
- board text added: "On"
- board text added: "Power"
- board text added: "Right"
- board text added: "Second"
- board text added: "Seconds"
- board text added: "Set Time"
- board text added: "Travel Time"
- board text added: "Unlock"
- board text added: "Up"
- board text added: "Year"

Commit message: a
Parts:
- SW9: value Set -> 12/24
Other:
- board text added: "12Hr"
- board text added: "24Hr"
Changed lines of the file:
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@@
 			)
 		)
-		(property "Value" "Set"
+		(property "Value" "12/24"
 			(at 0 3.81 0)
 			(layer "F.Fab")
@@
 	)
 	(gr_line
+		(start 63 131.5)
+		(end 63 130.5)
+		(stroke
+			(width 0.1)
+			(type default)
+		)
+		(layer "F.SilkS")
+	)
+	(gr_line
 		(start 131.25 161.25)
 		(end 124.25 161.25)
@@
 		(layer "F.SilkS")
 	)
+	(gr_line
+		(start 58 131.5)
+		(end 52.5 131.5)
+		(stroke
+			(width 0.1)
+			(type default)
+		)
+		(layer "F.SilkS")
+	)
 	(gr_arc
 		(start 119 142.25)
@@
 	)
 	(gr_line
+		(start 58 131.5)
+		(end 63 131.5)
+		(stroke
+			(width 0.1)
+			(type default)
+		)
+		(layer "F.SilkS")
+	)
+	(gr_line
 		(start 131.25 161.25)
 		(end 138.25 161.25)
@@
 	)
 	(gr_line
+		(start 52.5 131.5)
+		(end 52.5 130.5)
+		(stroke
+			(width 0.1)
+			(type default)
+		)
+		(layer "F.SilkS")
+	)
+	(gr_line
 		(start 138.25 161.25)
 		(end 138.25 162.25)
@@
 		)
 	)
+	(gr_text "24Hr"
+		(at 63 130 0)
+		(layer "F.SilkS")
+		(effects
+			(font
+				(size 1 1)
+				(thickness 0.1)
+			)
+			(justify bottom)
+		)
+	)
 	(gr_text "Lock\n"
 		(at 138.25 163.25 0)
@@
 		)
 	)
+	(gr_text "12Hr"
+		(at 52.5 130 0)
+		(layer "F.SilkS")
+		(effects
+			(font
+				(size 1 1)
+				(thickness 0.1)
+			)
+			(justify bottom)
+		)
+	)

Commit message: work
Parts:
- SW9: value 12/24 -> Set
Connections:
- net Mode renamed MODE
Changed lines of the file:
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@@
 	(net 218 "unconnected-(SW1-C-Pad3)")
 	(net 219 "unconnected-(SW9-C-Pad3)")
-	(net 220 "Mode")
+	(net 220 "MODE")
 	(footprint "Resistor_THT:R_Axial_DIN0207_L6.3mm_D2.5mm_P10.16mm_Horizontal"
 		(layer "F.Cu")
@@
 			(layers "*.Cu" "*.Mask")
 			(remove_unused_layers no)
-			(net 220 "Mode")
+			(net 220 "MODE")
 			(pinfunction "PD7")
 			(pintype "bidirectional")
@@
 			)
 		)
-		(property "Value" "12/24"
+		(property "Value" "Set"
 			(at 0 3.81 0)
 			(layer "F.Fab")
@@
 			(layers "*.Cu" "*.Mask")
 			(remove_unused_layers no)
-			(net 220 "Mode")
+			(net 220 "MODE")
 			(pinfunction "A")
 			(pintype "passive")
