File: new/clock.kicad_pcb (KiCad board)
At the start: 4 copper layers, 450 x 120 mm, 189 parts, among them J1 Barrel_Jack, J2 Conn_01x05_Socket, J3 Conn_PIC_ICSP_ICD, Q1 TIP127, Q10 2N3904, Q11 2N3904, Q12 2N3904, Q13 2N3904, Q14 2N3904, Q15 2N3904, Q16 2N3904, Q17 2N3904, Q18 2N3904, Q19 2N3904, Q2 TIP127, Q20 2N3904, Q21 2N3904, Q22 2N3904, Q23 2N3904, Q24 2N3904, Q25 2N3904, Q26 2N3904, Q27 2N3904, Q28 2N3904, Q29 2N3904, Q3 TIP127, Q30 2N3904, Q31 2N3904, Q32 2N3904, Q33 2N3904, Q34 2N3904, Q35 2N3904, Q36 2N3904, Q37 2N3904, Q38 2N3904, Q39 2N3904, Q4 TIP127, Q40 2N3904, Q41 2N3904, Q42 2N3904, Q43 2N3904, Q44 2N3904, Q45 2N3904, Q46 2N3904, Q5 TIP127, Q6 TIP127, Q7 TIP127, Q8 TIP127, Q9 2N3904, SW1 Power, SW2 Increment, SW3 Decrement, SW4 Up, SW5 Down, SW6 Left, SW7 Right, SW8 Set, SW9 Set, U1 ATmega328P-P, U2 74HC595, U3 74HC595, U4 74HC595, U5 74HC595, U6 74HC595, U7 74HC595, U8 DS1307+, Y1 16MHz, Y2 32.768kHz

Commit message: holes
Parts:
- added REF**: MountingHole_2.2mm_M2, MountingHole:MountingHole_2.2mm_M2, F.Cu at (101.2, 166.5)
- added REF**: MountingHole_2.2mm_M2, MountingHole:MountingHole_2.2mm_M2, F.Cu at (235.0, 127.5)
- added REF**: MountingHole_2.2mm_M2, MountingHole:MountingHole_2.2mm_M2, F.Cu at (496.5, 53.5)
- added REF**: MountingHole_2.2mm_M2, MountingHole:MountingHole_2.2mm_M2, F.Cu at (365.0, 127.5)
- added REF**: MountingHole_2.2mm_M2, MountingHole:MountingHole_2.2mm_M2, F.Cu at (53.5, 53.5)
- C3, C4, C5, C6, C7, C8, C9: footprint Capacitor_THT:C_Radial_D5.0mm_H11.0mm_P2.00mm -> Capacitor_THT:CP_Radial_D5.0mm_P2.00mm
- SW9: value Set -> 12/24

Commit message: revision number
Other:
- board text added: "Designed by Kyle Schmerge in association with UCSB IEEE www.github.com/kpzip www.ucsbieee.org Revision 1.0"
- board text removed: "Designed by Kyle Schmerge in association with UCSB IEEE. www.github.com/kpzip www.ucsbieee.org"
Changed lines of the file:
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@@
 		)
 	)
-	(gr_text "Designed by Kyle Schmerge in association with UCSB IEEE.\nwww.github.com/kpzip\nwww.ucsbieee.org"
-		(at 70.5 166.5 0)
+	(gr_text "Designed by Kyle Schmerge in association with UCSB IEEE\nwww.github.com/kpzip\nwww.ucsbieee.org\nRevision 1.0"
+		(at 70.5 168 0)
 		(layer "F.SilkS")
 		(effects

Commit message: avr isp
Parts:
- J3: value Conn_PIC_ICSP_ICD -> AVR_ISP
Changed lines of the file:
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@@
 			)
 		)
-		(property "Value" "Conn_PIC_ICSP_ICD"
+		(property "Value" "AVR_ISP"
 			(at 6.79 2.08 180)
 			(layer "F.Fab")
