File: new/clock.kicad_sch (KiCad schematic)
At the start: 186 parts, among them J1 Barrel_Jack, J2 Conn_01x05_Socket, J3 Conn_01x05_Pin, Q1 Q_PNP, Q10 2N3904, Q11 2N3904, Q12 2N3904, Q13 2N3904, Q14 2N3904, Q15 2N3904, Q16 2N3904, Q17 2N3904, Q18 2N3904, Q19 2N3904, Q2 Q_PNP, Q20 2N3904, Q21 2N3904, Q22 2N3904, Q23 2N3904, Q24 2N3904, Q25 2N3904, Q26 2N3904, Q27 2N3904, Q28 2N3904, Q29 2N3904, Q3 Q_PNP, Q30 2N3904, Q31 2N3904, Q32 2N3904, Q33 2N3904, Q34 2N3904, Q35 2N3904, Q36 2N3904, Q37 2N3904, Q38 2N3904, Q39 2N3904, Q4 Q_PNP, Q40 2N3904, Q41 2N3904, Q42 2N3904, Q43 2N3904, Q44 2N3904, Q45 2N3904, Q46 Q_PNP, Q5 Q_PNP, Q6 Q_PNP, Q7 Q_PNP, Q8 2N3904, Q9 2N3904, SW1 Increment, SW2 Decrement, SW3 Right, SW4 Left, SW5 Down, SW6 Up, SW7 Power, U1 ATmega328P-P, U2 74HC595, U3 74HC595, U4 74HC595, U5 74HC595, U6 74HC595, U7 74HC595, U8 DS1307+, Y1 16MHz, Y2 32.768kHz

Commit message: work
Parts:
- added D3: TVS, Diode_SMD:D_SMA_Handsoldering, symbol Device:D_Zener
- added J4: Conn_PIC_ICSP_ICD, symbol Connector:Conn_PIC_ICSP_ICD
- added SW8: Power, Button_Switch_THT:SW_Slide-03_Wuerth-WS-SLTV_10x2.5x6.4_P2.54mm, symbol Switch:SW_SPDT
- DS1, DS10, DS11, DS12, DS13, DS14, DS15, DS16, DS17, DS18, DS19, DS2, DS3, DS4, DS5, DS6, DS7, DS8, DS9: footprint Display_7Segment:DA56-11CGKWA -> Parts:DIPS2200W51P254L3580H1000Q18N
- J2: footprint Connector_PinSocket_1.00mm:PinSocket_1x04_P1.00mm_Vertical -> Connector_PinSocket_2.54mm:PinSocket_1x05_P2.54mm_Vertical
- J3: footprint Connector_PinHeader_1.00mm:PinHeader_1x04_P1.00mm_Vertical -> Connector_PinHeader_2.54mm:PinHeader_1x05_P2.54mm_Vertical
- Q1, Q2, Q3, Q4, Q5, Q6, Q7: value Q_PNP -> TIP127; symbol Device:Q_PNP -> Transistor_BJT:Q_PNP_BCE
- Q10: renamed from Q9; symbol Device:Q_NPN -> Transistor_BJT:Q_NPN_EBC
- Q11: renamed from Q10; symbol Device:Q_NPN -> Transistor_BJT:Q_NPN_EBC
- Q12: renamed from Q11; symbol Device:Q_NPN -> Transistor_BJT:Q_NPN_EBC
- Q13: renamed from Q12; symbol Device:Q_NPN -> Transistor_BJT:Q_NPN_EBC
- Q14: renamed from Q13; symbol Device:Q_NPN -> Transistor_BJT:Q_NPN_EBC
- Q15: renamed from Q14; symbol Device:Q_NPN -> Transistor_BJT:Q_NPN_EBC
- Q16: renamed from Q15; symbol Device:Q_NPN -> Transistor_BJT:Q_NPN_EBC
- Q17: renamed from Q16; symbol Device:Q_NPN -> Transistor_BJT:Q_NPN_EBC
- Q18: renamed from Q17; symbol Device:Q_NPN -> Transistor_BJT:Q_NPN_EBC
- Q19: renamed from Q18; symbol Device:Q_NPN -> Transistor_BJT:Q_NPN_EBC
- Q20: renamed from Q19; symbol Device:Q_NPN -> Transistor_BJT:Q_NPN_EBC
- Q21: renamed from Q20; symbol Device:Q_NPN -> Transistor_BJT:Q_NPN_EBC
- Q22: renamed from Q21; symbol Device:Q_NPN -> Transistor_BJT:Q_NPN_EBC
- Q23: renamed from Q22; symbol Device:Q_NPN -> Transistor_BJT:Q_NPN_EBC
- Q24: renamed from Q23; symbol Device:Q_NPN -> Transistor_BJT:Q_NPN_EBC
- Q25: renamed from Q24; symbol Device:Q_NPN -> Transistor_BJT:Q_NPN_EBC
- Q26: symbol Device:Q_NPN -> Transistor_BJT:Q_NPN_EBC
- Q27: renamed from Q28; symbol Device:Q_NPN -> Transistor_BJT:Q_NPN_EBC
- Q28: renamed from Q30; symbol Device:Q_NPN -> Transistor_BJT:Q_NPN_EBC
- Q29: renamed from Q32; symbol Device:Q_NPN -> Transistor_BJT:Q_NPN_EBC
- Q30: renamed from Q34; symbol Device:Q_NPN -> Transistor_BJT:Q_NPN_EBC
- Q31: renamed from Q36; symbol Device:Q_NPN -> Transistor_BJT:Q_NPN_EBC
- Q32: renamed from Q38; symbol Device:Q_NPN -> Transistor_BJT:Q_NPN_EBC
- Q33: renamed from Q25; symbol Device:Q_NPN -> Transistor_BJT:Q_NPN_EBC
- Q34: renamed from Q27; symbol Device:Q_NPN -> Transistor_BJT:Q_NPN_EBC
- Q35: renamed from Q29; symbol Device:Q_NPN -> Transistor_BJT:Q_NPN_EBC
- Q36: renamed from Q31; symbol Device:Q_NPN -> Transistor_BJT:Q_NPN_EBC
- Q37: renamed from Q33; symbol Device:Q_NPN -> Transistor_BJT:Q_NPN_EBC
- Q38: renamed from Q35; symbol Device:Q_NPN -> Transistor_BJT:Q_NPN_EBC
- Q39: renamed from Q37; symbol Device:Q_NPN -> Transistor_BJT:Q_NPN_EBC
- Q40: renamed from Q39; symbol Device:Q_NPN -> Transistor_BJT:Q_NPN_EBC
- Q41: renamed from Q40; symbol Device:Q_NPN -> Transistor_BJT:Q_NPN_EBC
- Q42: renamed from Q41; symbol Device:Q_NPN -> Transistor_BJT:Q_NPN_EBC
- Q43: renamed from Q42; symbol Device:Q_NPN -> Transistor_BJT:Q_NPN_EBC
- Q44: renamed from Q43; symbol Device:Q_NPN -> Transistor_BJT:Q_NPN_EBC
- Q45: renamed from Q44; symbol Device:Q_NPN -> Transistor_BJT:Q_NPN_EBC
- Q46: renamed from Q45; symbol Device:Q_NPN -> Transistor_BJT:Q_NPN_EBC
- Q8: renamed from Q46; value Q_PNP -> TIP127; symbol Device:Q_PNP -> Transistor_BJT:Q_PNP_BCE
- Q9: renamed from Q8; symbol Device:Q_NPN -> Transistor_BJT:Q_NPN_EBC
- SW7: value Power -> Set
Connections:
- net DIG_A: now also Q1.2 (C); no longer Q1.C
- net DIG_B: now also Q2.2 (C); no longer Q2.C
- net DIG_C: now also Q3.2 (C); no longer Q3.C
- net DIG_D: now also Q4.2 (C); no longer Q4.C
- net DIG_E: now also Q5.2 (C); no longer Q5.C
- net DIG_F: now also Q6.2 (C); no longer Q6.C
- net DIG_G: now also Q7.2 (C); no longer Q7.C
- net DP: now also Q8.2 (C); no longer Q8.C
- net GND: now also Q10.1 (E), Q11.1 (E), Q12.1 (E), Q13.1 (E), Q14.1 (E), Q15.1 (E), Q16.1 (E), Q17.1 (E), Q18.1 (E), Q19.1 (E), Q20.1 (E), Q21.1 (E), Q22.1 (E), Q23.1 (E), Q24.1 (E), Q25.1 (E), Q26.1 (E), Q27.1 (E), Q28.1 (E), Q29.1 (E), Q30.1 (E), Q31.1 (E), Q32.1 (E), Q33.1 (E), Q34.1 (E), Q35.1 (E), Q36.1 (E), Q37.1 (E), Q38.1 (E), Q39.1 (E), Q40.1 (E), Q41.1 (E), Q42.1 (E), Q43.1 (E), Q44.1 (E), Q45.1 (E), Q46.1 (E), Q9.1 (E), D3.2 (A), J4.3 (VSS); no longer Q10.E, Q11.E, Q12.E, Q13.E, Q14.E, Q15.E, Q16.E, Q17.E, Q18.E, Q19.E, Q20.E, Q21.E, Q22.E, Q23.E, Q24.E, Q25.E, Q26.E, Q27.E, Q28.E, Q29.E, Q30.E, Q31.E, Q32.E, Q33.E, Q34.E, Q35.E, Q36.E, Q37.E, Q38.E, Q39.E, Q40.E, Q41.E, Q42.E, Q43.E, Q44.E, Q45.E, Q46.E, Q9.E
- net VCC: now also Q1.3 (E), Q2.3 (E), Q3.3 (E), Q4.3 (E), Q5.3 (E), Q6.3 (E), Q7.3 (E), Q8.3 (E), D3.1 (K), J4.2 (VDD), SW8.1 (A); no longer J1.1, Q1.E, Q2.E, Q3.E, Q4.E, Q5.E, Q6.E, Q7.E, Q8.E
- net at R7.2: now also Q7.1 (B); no longer Q7.B
- net at R1.2: now also Q1.1 (B); no longer Q1.B
- net at R31.2: now also Q20.2 (B); no longer Q20.B
- net at R63.2: now also Q36.2 (B); no longer Q36.B
- net at R64.2: now also Q36.3 (C); no longer Q36.C
- net at R25.2: now also Q17.2 (B); no longer Q17.B
- net at R41.2: now also Q25.2 (B); no longer Q25.B
- net at R42.2: now also Q25.3 (C); no longer Q25.C
- net at R33.2: now also Q21.2 (B); no longer Q21.B
- net at R34.2: now also Q21.3 (C); no longer Q21.C
- net at R79.2: now also Q44.2 (B); no longer Q44.B
- net at R80.2: now also Q44.3 (C); no longer Q44.C
- net at R51.2: now also Q30.2 (B); no longer Q30.B
- net at R52.2: now also Q30.3 (C); no longer Q30.C
- net at R55.2: now also Q32.2 (B); no longer Q32.B
- net at R56.2: now also Q32.3 (C); no longer Q32.C
- net at R60.2: now also Q34.3 (C); no longer Q34.C
- net at R26.2: now also Q17.3 (C); no longer Q17.C
- net at R40.2: now also Q24.3 (C); no longer Q24.C
- net at R72.2: now also Q40.3 (C); no longer Q40.C
- net at R47.2: now also Q28.2 (B); no longer Q28.B
- net at R48.2: now also Q28.3 (C); no longer Q28.C
- net at R18.2: now also Q13.3 (C); no longer Q13.C
- net at R75.2: now also Q42.2 (B); no longer Q42.B
- net at R76.2: now also Q42.3 (C); no longer Q42.C
- net at R22.2: now also Q15.3 (C); no longer Q15.C
- net at R71.2: now also Q40.2 (B); no longer Q40.B
- net at R17.2: now also Q13.2 (B); no longer Q13.B
- net at R43.2: now also Q26.2 (B); no longer Q26.B
- net at R19.2: now also Q14.2 (B); no longer Q14.B
- net at R20.2: now also Q14.3 (C); no longer Q14.C
- net at R6.2: now also Q6.1 (B); no longer Q6.B
- net at R36.2: now also Q22.3 (C); no longer Q22.C
- net at R4.2: now also Q4.1 (B); no longer Q4.B
- net at R66.2: now also Q37.3 (C); no longer Q37.C
- net at R14.2: now also Q11.3 (C); no longer Q11.C
- net at R83.2: now also Q46.2 (B); no longer Q46.B
- net at R84.2: now also Q46.3 (C); no longer Q46.C
- net at R57.2: now also Q33.2 (B); no longer Q33.B
- net at R77.2: now also Q43.2 (B); no longer Q43.B
- net at R32.2: now also Q20.3 (C); no longer Q20.C
- net at R58.2: now also Q33.3 (C); no longer Q33.C
- net at R78.2: now also Q43.3 (C); no longer Q43.C
- net at R21.2: now also Q15.2 (B); no longer Q15.B
- net at R45.2: now also Q27.2 (B); no longer Q27.B
- net at R24.2: now also Q16.3 (C); no longer Q16.C
- net at R70.2: now also Q39.3 (C); no longer Q39.C
- net at R74.2: now also Q41.3 (C); no longer Q41.C
- net at R46.2: now also Q27.3 (C); no longer Q27.C
- net at R23.2: now also Q16.2 (B); no longer Q16.B
- net at R54.2: now also Q31.3 (C); no longer Q31.C
- net at R44.2: now also Q26.3 (C); no longer Q26.C
- net at R61.2: now also Q35.2 (B); no longer Q35.B
- net at R81.2: now also Q45.2 (B); no longer Q45.B
- net at R82.2: now also Q45.3 (C); no longer Q45.C
- net at R67.2: now also Q38.2 (B); no longer Q38.B
- net at R68.2: now also Q38.3 (C); no longer Q38.C
- net at R11.2: now also Q10.2 (B); no longer Q10.B
- net at R12.2: now also Q10.3 (C); no longer Q10.C
- net at R13.2: now also Q11.2 (B); no longer Q11.B
- net at R15.2: now also Q12.2 (B); no longer Q12.B
- net at R16.2: now also Q12.3 (C); no longer Q12.C
- net at R62.2: now also Q35.3 (C); no longer Q35.C
- net at R10.2: now also Q9.3 (C); no longer Q9.C
- net at R27.2: now also Q18.2 (B); no longer Q18.B
- net at R28.2: now also Q18.3 (C); no longer Q18.C
- net at R39.2: now also Q24.2 (B); no longer Q24.B
- net at R73.2: now also Q41.2 (B); no longer Q41.B
- net at R49.2: now also Q29.2 (B); no longer Q29.B
- net at R50.2: now also Q29.3 (C); no longer Q29.C
- net at R53.2: now also Q31.2 (B); no longer Q31.B
- net at R9.2: now also Q9.2 (B); no longer Q9.B
- net at R3.2: now also Q3.1 (B); no longer Q3.B
- net at R69.2: now also Q39.2 (B); no longer Q39.B
- net at R2.2: now also Q2.1 (B); no longer Q2.B
- net at R35.2: now also Q22.2 (B); no longer Q22.B
- net at R37.2: now also Q23.2 (B); no longer Q23.B
- net at R65.2: now also Q37.2 (B); no longer Q37.B
- net at R38.2: now also Q23.3 (C); no longer Q23.C
- net at R59.2: now also Q34.2 (B); no longer Q34.B
- net at R29.2: now also Q19.2 (B); no longer Q19.B
- net at R8.2: now also Q8.1 (B); no longer Q8.B
- net at R5.2: now also Q5.1 (B); no longer Q5.B
- net at R30.2: now also Q19.3 (C); no longer Q19.C
- new net: J1.1, SW8.2 (B)
- no-connect marks 10 -> 11

Commit message: huge
Connections:
- net DS37: now also DS19.13 (DIG2_CC)
Changed lines of the file:
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@@
+	(wire
+		(pts
+			(xy 320.04 492.76) (xy 325.12 492.76)
+		)
+		(stroke
+			(width 0)
+			(type default)
+		)
+	)
 	(wire
 		(pts

Commit message: almost
Parts:
- J4: footprint (none) -> Connector_IDC:IDC-Header_2x03_P2.54mm_Vertical; symbol Connector:Conn_PIC_ICSP_ICD -> Connector:AVR-ISP-6
Connections:
- net GND: now also J4.6 (GND); no longer J4.3 (VSS)
- net RCLK: now also J4.4 (MOSI)
- net SER: now also J4.1 (MISO)
- net RESET: now reaches U1.1 (~{RESET}/PC6)
- net RESET: now also J4.5 (~{RST})
- net SCK: now reaches U1.19 (PB5)
- net SCK: now also J4.3 (SCK)
- no-connect marks 11 -> 9
Changed lines of the file:
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@@
 	)
 	(no_connect
+		(at 308.61 323.85)
+	)
+	(no_connect
 		(at 382.27 264.16)
 	)
@@
 	)
 	(no_connect
-		(at 308.61 323.85)
-	)
-	(no_connect
 		(at 382.27 299.72)
 	)
-	(no_connect
-		(at 382.27 276.86)
-	)
-	(no_connect
-		(at 382.27 251.46)
-	)
 	(wire
 		(pts
@@
 	(wire
 		(pts
-			(xy 443.23 302.26) (xy 443.23 306.07)
+			(xy 445.77 302.26) (xy 445.77 306.07)
 		)
 		(stroke
@@
 	(wire
 		(pts
+			(xy 382.27 251.46) (xy 387.35 251.46)
+		)
+		(stroke
+			(width 0)
+			(type default)
+		)
+	)
+	(wire
+		(pts
 			(xy 217.17 208.28) (xy 217.17 213.36)
 		)
@@
 	(wire
 		(pts
+			(xy 458.47 289.56) (xy 464.82 289.56)
+		)
+		(stroke
+			(width 0)
+			(type default)
+		)
+	)
+	(wire
+		(pts
 			(xy 565.15 480.06) (xy 570.23 480.06)
 		)
@@
 	(wire
 		(pts
+			(xy 458.47 292.1) (xy 464.82 292.1)
+		)
+		(stroke
+			(width 0)
+			(type default)
+		)
+	)
+	(wire
+		(pts
 			(xy 289.56 441.96) (xy 294.64 441.96)
 		)
@@
 	(wire
 		(pts
+			(xy 458.47 294.64) (xy 464.82 294.64)
+		)
+		(stroke
+			(width 0)
+			(type default)
+		)
+	)
+	(wire
+		(pts
 			(xy 166.37 115.57) (xy 166.37 119.38)
 		)
@@
 	(wire
 		(pts
+			(xy 458.47 287.02) (xy 464.82 287.02)
+		)
+		(stroke
+			(width 0)
+			(type default)
+		)
+	)
+	(wire
+		(pts
 			(xy 617.22 345.44) (xy 615.95 345.44)
 		)
@@
 	(wire
 		(pts
-			(xy 443.23 278.13) (xy 443.23 281.94)
+			(xy 445.77 275.59) (xy 445.77 279.4)
 		)
 		(stroke
@@
 	(wire
 		(pts
+			(xy 382.27 276.86) (xy 387.35 276.86)
+		)
+		(stroke
+			(width 0)
+			(type default)
+		)
+	)
+	(wire
+		(pts
 			(xy 312.42 222.25) (xy 312.42 236.22)
 		)
@@
 	(global_label "RCLK"
 		(shape input)
+		(at 464.82 289.56 0)
+		(fields_autoplaced yes)
+		(effects
+			(font
+				(size 1.27 1.27)
+			)
+			(justify left)
+		)
+		(property "Intersheetrefs" "${INTERSHEET_REFS}"
+			(at 472.6433 289.56 0)
+			(effects
+				(font
+					(size 1.27 1.27)
+				)
+				(justify left)
+				(hide yes)
+			)
+		)
+	)
+	(global_label "RCLK"
+		(shape input)
 		(at 281.94 161.29 180)
 		(fields_autoplaced yes)
@@
 		)
 	)
+	(global_label "RESET"
+		(shape input)
+		(at 464.82 294.64 0)
+		(fields_autoplaced yes)
+		(effects
+			(font
+				(size 1.27 1.27)
+			)
+			(justify left)
+		)
+		(property "Intersheetrefs" "${INTERSHEET_REFS}"
+			(at 473.5503 294.64 0)
+			(effects
+				(font
+					(size 1.27 1.27)
+				)
+				(justify left)
+				(hide yes)
+			)
+		)
+	)
 	(global_label "DP"
 		(shape input)
@@
 		)
 	)
+	(global_label "SCK"
+		(shape input)
+		(at 464.82 292.1 0)
+		(fields_autoplaced yes)
+		(effects
+			(font
+				(size 1.27 1.27)
+			)
+			(justify left)
+		)
+		(property "Intersheetrefs" "${INTERSHEET_REFS}"
+			(at 471.5547 292.1 0)
+			(effects
+				(font
+					(size 1.27 1.27)
+				)
+				(justify left)
+				(hide yes)
+			)
+		)
+	)
 	(global_label "DIG_B"
 		(shape input)
@@
 		)
 	)
+	(global_label "SCK"
+		(shape input)
+		(at 387.35 251.46 0)
+		(fields_autoplaced yes)
+		(effects
+			(font
+				(size 1.27 1.27)
+			)
+			(justify left)
+		)
+		(property "Intersheetrefs" "${INTERSHEET_REFS}"
+			(at 394.0847 251.46 0)
+			(effects
+				(font
+					(size 1.27 1.27)
+				)
+				(justify left)
+				(hide yes)
+			)
+		)
+	)
 	(global_label "DIG_F"
 		(shape input)
@@
 		)
 	)
+	(global_label "SER"
+		(shape input)
+		(at 464.82 287.02 0)
+		(fields_autoplaced yes)
+		(effects
+			(font
+				(size 1.27 1.27)
+			)
+			(justify left)
+		)
+		(property "Intersheetrefs" "${INTERSHEET_REFS}"
+			(at 471.4337 287.02 0)
+			(effects
+				(font
+					(size 1.27 1.27)
+				)
+				(justify left)
+				(hide yes)
+			)
+		)
+	)
 	(global_label "DIG_F"
 		(shape input)
@@
 		)
 	)
+	(global_label "RESET"
+		(shape input)
+		(at 387.35 276.86 0)
+		(fields_autoplaced yes)
+		(effects
+			(font
+				(size 1.27 1.27)
+			)
+			(justify left)
+		)
+		(property "Intersheetrefs" "${INTERSHEET_REFS}"
+			(at 396.0803 276.86 0)
+			(effects
+				(font
+					(size 1.27 1.27)
+				)
+				(justify left)
+				(hide yes)
+			)
+		)
+	)
 	(global_label "DP"
 		(shape input)
@@
 	(symbol
 		(lib_id "power:GND")
-		(at 443.23 306.07 0)
+		(at 445.77 306.07 0)
 		(unit 1)
 		(exclude_from_sim no)
@@
 		(fields_autoplaced yes)
 		(property "Reference" "#PWR088"
-			(at 443.23 312.42 0)
+			(at 445.77 312.42 0)
 			(effects
 				(font
@@
 		)
 		(property "Value" "GND"
-			(at 443.23 311.15 0)
+			(at 445.77 311.15 0)
 			(effects
 				(font
@@
 		)
 		(property "Footprint" ""
-			(at 443.23 306.07 0)
+			(at 445.77 306.07 0)
 			(effects
 				(font
@@
 		)
 		(property "Datasheet" ""
-			(at 443.23 306.07 0)
+			(at 445.77 306.07 0)
 			(effects
 				(font
@@
 		)
 		(property "Description" "Power symbol creates a global label with name \"GND\" , ground"
-			(at 443.23 306.07 0)
+			(at 445.77 306.07 0)
 			(effects
 				(font
@@
 	(symbol
 		(lib_id "power:VCC")
-		(at 443.23 278.13 0)
+		(at 445.77 275.59 0)
 		(unit 1)
 		(exclude_from_sim no)
@@
 		(dnp no)
 		(property "Reference" "#PWR087"
-			(at 443.23 281.94 0)
+			(at 445.77 279.4 0)
 			(effects
 				(font
@@
 		)
 		(property "Value" "VCC"
-			(at 443.23 274.066 0)
+			(at 445.77 271.526 0)
 			(effects
 				(font
@@
 		)
 		(property "Footprint" ""
-			(at 443.23 278.13 0)
+			(at 445.77 275.59 0)
 			(effects
 				(font
@@
 		)
 		(property "Datasheet" ""
-			(at 443.23 278.13 0)
+			(at 445.77 275.59 0)
 			(effects
 				(font
@@
 		)
 		(property "Description" "Power symbol creates a global label with name \"VCC\""
-			(at 443.23 278.13 0)
+			(at 445.77 275.59 0)
 			(effects
 				(font
@@
 	)
 	(symbol
-		(lib_id "Connector:Conn_PIC_ICSP_ICD")
+		(lib_id "Connector:AVR-ISP-6")
 		(at 448.31 292.1 0)
 		(unit 1)
@@
 		(on_board yes)
 		(dnp no)
-		(fields_autoplaced yes)
 		(property "Reference" "J4"
-			(at 439.42 290.8299 0)
+			(at 439.42 289.5599 0)
 			(effects
 				(font
@@
 		)
 		(property "Value" "Conn_PIC_ICSP_ICD"
-			(at 439.42 293.3699 0)
+			(at 466.852 302.768 0)
 			(effects
 				(font
@@
 			)
 		)
-		(property "Footprint" ""
-			(at 449.58 288.29 0)
+		(property "Footprint" "Connector_IDC:IDC-Header_2x03_P2.54mm_Vertical"
+			(at 441.96 290.83 90)
 			(effects
 				(font
@@
 			)
 		)
-		(property "Datasheet" "http://ww1.microchip.com/downloads/en/devicedoc/30277d.pdf"
-			(at 440.69 295.91 90)
+		(property "Datasheet" "~"
+			(at 415.925 306.07 0)
 			(effects
 				(font
@@
 			)
 		)
-		(property "Description" "Microchip PIC In-Circuit Serial Programming/Debugging (ICSP/ICD) connector"
+		(property "Description" "Atmel 6-pin ISP connector"
 			(at 448.31 292.1 0)
 			(effects

Commit message: done?
Parts:
- removed J3: Conn_01x05_Pin, Connector_PinHeader_2.54mm:PinHeader_1x05_P2.54mm_Vertical, symbol Connector:Conn_01x05_Pin
- added SW9: Set, Button_Switch_THT:SW_Slide-03_Wuerth-WS-SLTV_10x2.5x6.4_P2.54mm, symbol Switch:SW_SPDT
- renumbered J4 to J3, SW8 to SW1, SW1 to SW2, SW2 to SW3, SW6 to SW4, SW4 to SW6, SW3 to SW7, SW7 to SW8
Connections:
- net GND: now also B1.2 (-), U8.4 (GND), SW9.2 (B)
- net SCL: now also U8.6 (SCL)
- net SDA: now also U8.5 (SDA)
- net VCC: now also U8.8 (VCC)
- net Mode: now reaches U1.13 (PD7)
- net Mode: now also SW9.1 (A)
- no-connect marks 9 -> 10
Other:
- moved on the sheet: B1, J2, U8, Y2

Commit message: work
Connections:
- net Mode renamed MODE
Changed lines of the file:
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@@
 		)
 	)
-	(global_label "Mode"
+	(global_label "MODE"
 		(shape input)
 		(at 387.35 299.72 0)
@@
 		)
 		(property "Intersheetrefs" "${INTERSHEET_REFS}"
-			(at 395.1732 299.72 0)
+			(at 395.5361 299.72 0)
 			(effects
 				(font
@@
 		)
 	)
-	(global_label "Mode"
+	(global_label "MODE"
 		(shape input)
 		(at 581.66 222.25 0)
@@
 		)
 		(property "Intersheetrefs" "${INTERSHEET_REFS}"
-			(at 589.4832 222.25 0)
-			(effects
-				(font
+			(at 589.8461 222.25 0)
+			(effects
+				(font

Commit message: holes
Parts:
- C3, C4, C5, C6, C7, C8, C9: footprint Capacitor_THT:C_Radial_D5.0mm_H11.0mm_P2.00mm -> Capacitor_THT:CP_Radial_D5.0mm_P2.00mm
- SW9: value Set -> 12/24
Changed lines of the file:
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@@
 			)
 		)
-		(property "Footprint" "Capacitor_THT:C_Radial_D5.0mm_H11.0mm_P2.00mm"
+		(property "Footprint" "Capacitor_THT:CP_Radial_D5.0mm_P2.00mm"
 			(at 48.26 162.56 0)
 			(effects
@@
 			)
 		)
-		(property "Footprint" "Capacitor_THT:C_Radial_D5.0mm_H11.0mm_P2.00mm"
+		(property "Footprint" "Capacitor_THT:CP_Radial_D5.0mm_P2.00mm"
 			(at 49.53 320.04 0)
 			(effects
@@
 			)
 		)
-		(property "Value" "Set"
+		(property "Value" "12/24"
 			(at 570.23 218.44 0)
 			(effects
@@
 			)
 		)
-		(property "Footprint" "Capacitor_THT:C_Radial_D5.0mm_H11.0mm_P2.00mm"
+		(property "Footprint" "Capacitor_THT:CP_Radial_D5.0mm_P2.00mm"
 			(at 48.26 110.49 0)
 			(effects
@@
 			)
 		)
-		(property "Footprint" "Capacitor_THT:C_Radial_D5.0mm_H11.0mm_P2.00mm"
+		(property "Footprint" "Capacitor_THT:CP_Radial_D5.0mm_P2.00mm"
 			(at 49.53 267.97 0)
 			(effects
@@
 			)
 		)
-		(property "Footprint" "Capacitor_THT:C_Radial_D5.0mm_H11.0mm_P2.00mm"
+		(property "Footprint" "Capacitor_THT:CP_Radial_D5.0mm_P2.00mm"
 			(at 49.53 215.9 0)
 			(effects
@@
 			)
 		)
-		(property "Footprint" "Capacitor_THT:C_Radial_D5.0mm_H11.0mm_P2.00mm"
+		(property "Footprint" "Capacitor_THT:CP_Radial_D5.0mm_P2.00mm"
 			(at 48.26 40.64 0)
 			(effects
@@
 			)
 		)
-		(property "Footprint" "Capacitor_THT:C_Radial_D5.0mm_H11.0mm_P2.00mm"
+		(property "Footprint" "Capacitor_THT:CP_Radial_D5.0mm_P2.00mm"
 			(at 349.25 233.68 0)
 			(effects

Commit message: avr isp
Parts:
- J3: value Conn_PIC_ICSP_ICD -> AVR_ISP
Changed lines of the file:
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@@
 			)
 		)
-		(property "Value" "Conn_PIC_ICSP_ICD"
-			(at 466.852 302.768 0)
+		(property "Value" "AVR_ISP"
+			(at 456.692 302.006 0)
 			(effects
 				(font
