File: new/pcb/1.0/clock.kicad_sch (KiCad schematic)
At the start: 189 parts, among them J1 Barrel_Jack, J2 Conn_01x05_Socket, J3 AVR_ISP, Q1 TIP127, Q10 2N3904, Q11 2N3904, Q12 2N3904, Q13 2N3904, Q14 2N3904, Q15 2N3904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

Commit message: set title
Other:
- title: (none) -> IEEE Clock
Changed lines of the file:
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@@
 	(generator_version "9.0")
 	(paper "A1")
+	(title_block
+		(title "IEEE Clock")
+		(date "2025-05-08")
+		(rev "1.0")
+	)
 	(junction
 		(at 251.46 46.99)
