File: new/pcb/clock.kicad_pcb (KiCad board)
At the start: 4 copper layers, 450 x 120 mm, 194 parts, among them J1 Barrel_Jack, J2 Conn_01x05_Socket, J3 AVR_ISP, Q1 TIP127, Q10 2N3904, Q11 2N3904, Q12 2N3904, Q13 2N3904, Q14 2N3904, Q15 2N3904, Q16 2N3904, Q17 2N3904, Q18 2N3904, Q19 2N3904, Q2 TIP127, Q20 2N3904, Q21 2N3904, Q22 2N3904, Q23 2N3904, Q24 2N3904, Q25 2N3904, Q26 2N3904, Q27 2N3904, Q28 2N3904, Q29 2N3904, Q3 TIP127, Q30 2N3904, Q31 2N3904, Q32 2N3904, Q33 2N3904, Q34 2N3904, Q35 2N3904, Q36 2N3904, Q37 2N3904, Q38 2N3904, Q39 2N3904, Q4 TIP127, Q40 2N3904, Q41 2N3904, Q42 2N3904, Q43 2N3904, Q44 2N3904, Q45 2N3904, Q46 2N3904, Q5 TIP127, Q6 TIP127, Q7 TIP127, Q8 TIP127, Q9 2N3904, SW1 Power, SW2 Increment, SW3 Decrement, SW4 Up, SW5 Down, SW6 Left, SW7 Right, SW8 Set, SW9 12/24, U1 ATmega328P-P, U2 74HC595, U3 74HC595, U4 74HC595, U5 74HC595, U6 74HC595, U7 74HC595, U8 DS1307+, Y1 16MHz, Y2 32.768kHz

Commit message: run it back
Parts:
- removed H1, H2, H3, H4, H5: Hole, MountingHole:MountingHole_2.2mm_M2_ISO7380_Pad
- added C10: 100nF, Capacitor_SMD:C_1206_3216Metric_Pad1.33x1.80mm_HandSolder, F.Cu at (480.8, 143.0)
- added REF**: MountingHole_2.2mm_M2, MountingHole:MountingHole_2.2mm_M2, F.Cu at (101.2, 166.5)
- added REF**: MountingHole_2.2mm_M2, MountingHole:MountingHole_2.2mm_M2, F.Cu at (235.0, 127.5)
- added REF**: MountingHole_2.2mm_M2, MountingHole:MountingHole_2.2mm_M2, F.Cu at (496.5, 53.5)
- added REF**: MountingHole_2.2mm_M2, MountingHole:MountingHole_2.2mm_M2, F.Cu at (365.0, 127.5)
- added REF**: MountingHole_2.2mm_M2, MountingHole:MountingHole_2.2mm_M2, F.Cu at (53.5, 53.5)
Connections:
- J3 pad 4: ~{SRCLR} -> RCLK
- U1 pad 17: ~{SRCLR} -> RCLK
- U1 pad 21: GND -> Net-(U1-AREF)
- U2 pad 10: ~{SRCLR} -> VCC
- U2 pad 12: GND -> RCLK
- U3 pad 10: ~{SRCLR} -> VCC
- U3 pad 12: GND -> RCLK
- U4 pad 10: ~{SRCLR} -> VCC
- U4 pad 12: GND -> RCLK
- U5 pad 10: ~{SRCLR} -> VCC
- U5 pad 12: GND -> RCLK
- U6 pad 10: ~{SRCLR} -> VCC
- U6 pad 12: GND -> RCLK
- U7 pad 10: ~{SRCLR} -> VCC
- U7 pad 12: GND -> RCLK
Routing:
- net RCLK: track 0.00 -> 201.8 mm
- net ~{SRCLR}: track 151.1 -> 0.00 mm, vias 2 -> 0
- net Net-(U1-AREF): track 0.00 -> 64.4 mm, vias 0 -> 3
- net CTRL_DS17: vias 2 -> 1
Other:
- board text added: "Designed by Kyle Schmerge in association with UCSB IEEE www.github.com/kpzip www.ucsbieee.org Revision 1.0"
- board text removed: "5V Input"
- board text removed: "Designed by Kyle Schmerge in association with UCSB IEEE www.github.com/kpzip www.ucsbieee.org Revision 1.1"

Commit message: Re add fixes
Parts:
- removed REF** (x5): MountingHole_2.2mm_M2, MountingHole:MountingHole_2.2mm_M2
- added H1: Hole, MountingHole:MountingHole_2.2mm_M2_ISO7380_Pad, F.Cu at (53.5, 53.5)
- added H2: Hole, MountingHole:MountingHole_2.2mm_M2_ISO7380_Pad, F.Cu at (496.5, 53.5)
- added H3: Hole, MountingHole:MountingHole_2.2mm_M2_ISO7380_Pad, F.Cu at (365.0, 127.6)
- added H4: Hole, MountingHole:MountingHole_2.2mm_M2_ISO7380_Pad, F.Cu at (235.2, 127.8)
- added H5: Hole, MountingHole:MountingHole_2.2mm_M2_ISO7380_Pad, F.Cu at (101.2, 166.4)
Routing:
- net CTRL_DS17: track 107.7 -> 110.0 mm, vias 1 -> 0
- net Net-(U1-AREF): track 64.4 -> 66.0 mm
Other:
- board text added: "5V Input"

Commit message: logo
Parts:
- added LG1: Logo_Open_Hardware_Small, Parts:UCSB_IEEE_Logo, F.Cu at (147.4, 161.8)
Other:
- board text added: "Designed by Kyle Schmerge in association with UCSB IEEE www.github.com/kpzip www.ucsbieee.org Revision 1.1"
- board text removed: "Designed by Kyle Schmerge in association with UCSB IEEE www.github.com/kpzip www.ucsbieee.org Revision 1.0"
