File: new/pcb/clock.kicad_sch (KiCad schematic)
At the start: 194 parts, among them J1 Barrel_Jack, J2 Conn_01x05_Socket, J3 AVR_ISP, Q1 TIP127, Q10 2N3904, Q11 2N3904, Q12 2N3904, Q13 2N3904, Q14 2N3904, Q15 2N3904, Q16 2N3904, Q17 2N3904, Q18 2N3904, Q19 2N3904, Q2 TIP127, Q20 2N3904, Q21 2N3904, Q22 2N3904, Q23 2N3904, Q24 2N3904, Q25 2N3904, Q26 2N3904, Q27 2N3904, Q28 2N3904, Q29 2N3904, Q3 TIP127, Q30 2N3904, Q31 2N3904, Q32 2N3904, Q33 2N3904, Q34 2N3904, Q35 2N3904, Q36 2N3904, Q37 2N3904, Q38 2N3904, Q39 2N3904, Q4 TIP127, Q40 2N3904, Q41 2N3904, Q42 2N3904, Q43 2N3904, Q44 2N3904, Q45 2N3904, Q46 2N3904, Q5 TIP127, Q6 TIP127, Q7 TIP127, Q8 TIP127, Q9 2N3904, SW1 Power, SW2 Increment, SW3 Decrement, SW4 Up, SW5 Down, SW6 Left, SW7 Right, SW8 Set, SW9 12/24, U1 ATmega328P-P, U2 74HC595, U3 74HC595, U4 74HC595, U5 74HC595, U6 74HC595, U7 74HC595, U8 DS1307+, Y1 16MHz, Y2 32.768kHz

Commit message: run it back
Parts:
- removed H1, H2, H3, H4, H5: Hole, MountingHole:MountingHole_2.2mm_M2_ISO7380_Pad, symbol Mechanical:MountingHole_Pad
- added C10: 100nF, Capacitor_SMD:C_1206_3216Metric_Pad1.33x1.80mm_HandSolder, symbol Device:C
Connections:
- net GND: now also C10.2; no longer U1.21 (AREF), U2.12 (RCLK), U3.12 (RCLK), U4.12 (RCLK), U5.12 (RCLK), U6.12 (RCLK), U7.12 (RCLK)
- net VCC: now also U2.10 (~{SRCLR}), U3.10 (~{SRCLR}), U4.10 (~{SRCLR}), U5.10 (~{SRCLR}), U6.10 (~{SRCLR}), U7.10 (~{SRCLR})
- removed net ~{SRCLR}: J3.4 (MOSI), U1.17 (PB3), U2.10 (~{SRCLR}), U3.10 (~{SRCLR}), U4.10 (~{SRCLR}), U5.10 (~{SRCLR}), U6.10 (~{SRCLR}), U7.10 (~{SRCLR})
- new net: C10.1, U1.21 (AREF)
- new net RCLK: J3.4 (MOSI), U1.17 (PB3), U2.12 (RCLK), U3.12 (RCLK), U4.12 (RCLK), U5.12 (RCLK), U6.12 (RCLK), U7.12 (RCLK)
Other:
- moved on the sheet: C3

Commit message: Re add fixes
Parts:
- added H1, H2, H3, H4, H5: Hole, MountingHole:MountingHole_2.2mm_M2_ISO7380_Pad, symbol Mechanical:MountingHole_Pad
Connections:
- net GND: now also H1.1, H2.1, H3.1, H4.1, H5.1

Commit message: set title
Other:
- title: (none) -> IEEE Clock
Changed lines of the file:
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@@
 	(generator_version "9.0")
 	(paper "A1")
+	(title_block
+		(title "IEEE Clock")
+		(date "2025-06-01")
+		(rev "1.1")
+	)
 	(junction
 		(at 411.48 281.94)

Commit message: logo
Parts:
- added LG1: Logo_Open_Hardware_Small, Parts:UCSB_IEEE_Logo, symbol Graphic:Logo_Open_Hardware_Small
Changed lines of the file:
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@@
+	)
+	(symbol
+		(lib_id "Graphic:Logo_Open_Hardware_Small")
+		(at 707.39 565.15 0)
+		(unit 1)
+		(exclude_from_sim no)
+		(in_bom no)
+		(on_board yes)
+		(dnp no)
+		(fields_autoplaced yes)
+		(property "Reference" "LG1"
+			(at 707.39 558.165 0)
+			(effects
+				(font
+					(size 1.27 1.27)
+				)
+				(hide yes)
+			)
+		)
+		(property "Value" "Logo_Open_Hardware_Small"
+			(at 707.39 570.865 0)
+			(effects
+				(font
+					(size 1.27 1.27)
+				)
+				(hide yes)
+			)
+		)
+		(property "Footprint" "Parts:UCSB_IEEE_Logo"
+			(at 707.39 565.15 0)
+			(effects
+				(font
+					(size 1.27 1.27)
+				)
+				(hide yes)
+			)
+		)
+		(property "Datasheet" "~"
+			(at 707.39 565.15 0)
+			(effects
+				(font
+					(size 1.27 1.27)
+				)
+				(hide yes)
+			)
+		)
+		(property "Description" "Open Hardware logo, small"
+			(at 707.39 565.15 0)
+			(effects
+				(font
+					(size 1.27 1.27)
+				)
+				(hide yes)
+			)
+		)
+		(property "Sim.Enable" "0"
+			(at 707.39 565.15 0)
+			(effects
+				(font
+					(size 1.27 1.27)
+				)
+				(hide yes)
+			)
+		)
+		(instances
+			(project ""
+				(path "/81fe6255-7db2-4e1e-90bf-860defad696b"
+					(reference "LG1")
+					(unit 1)
+				)
+			)
+		)
 	)
 	(symbol
